File: In Development/PCB Designs/BrakeLightBoard/brakelight.sch (EAGLE design)
At the start: 11 parts, among them IC1 LM311N, IC2 LM311N, Q1 SUP75N06-08, Q2 SUP75N06-08

Commit message: Updated brakelight board schematic and board
Parts:
- removed TRIMPOT: (no value), resistor:R-TRIMM74W
- added ARDUINO_READ: 1751248, con-phoenix-350:1751248
- added LIPO_CONN: (no value), con-wago-500:W237-102
- added TRIMPOT1, TRIMPOT2: (no value), bourns:3386-Y
- Q1, Q2: value SUP75N06-08 -> 75N06
Connections:
- removed net THRESH: IC1.+IN, IC2.+IN, TRIMPOT.S
- new net THRESH1: IC1.+IN, TRIMPOT1.2
- new net THRESH2: IC2.+IN, TRIMPOT2.2
- net 5V: now also TRIMPOT1.1, TRIMPOT2.1; no longer TRIMPOT.A
- net GND: now also LIPO_CONN-2.KL, TRIMPOT1.3, TRIMPOT2.3; no longer TRIMPOT.E
- net N$1: now also R1.1; no longer R2.1
- net N$2: now also R2.1; no longer R1.1
- net VCC: now also LIPO_CONN-1.KL
Other:
- moved on the sheet: 5V_LINREG, R1, R2

Commit message: Revised brakelight schematic
Parts:
- removed ARDUINO_READ: 1751248, con-phoenix-350:1751248
- added INO_READ: (no value), con-wago-500:W237-102
Connections:
- net PT1: now also INO_READ-1.KL
- net PT2: now also INO_READ-2.KL

Commit message: Finished BrakeLight Board
Parts:
- removed IC1, IC2: LM311N, linear:LM311N
- added U$1, U$2: LM311, GTOR:LM311
Connections:
- net 5V: now also U$1.V+, U$2.V+; no longer IC1.V+, IC2.V+
- net GND: now also U$1.GND, U$2.GND; no longer IC1.GND, IC2.GND
- net N$1: now also U$1.OUT; no longer IC1.OUT
- net N$2: now also U$2.OUT; no longer IC2.OUT
- net PT1: now also U$1.-IN; no longer IC1.-IN
- net PT2: now also U$2.-IN; no longer IC2.-IN
- net THRESH1: now also U$1.+IN; no longer IC1.+IN
- net THRESH2: now also U$2.+IN; no longer IC2.+IN
