File: Dashboard/Circuitry/DashDial.sch (EAGLE design)
At the start: 33 parts, among them IC1 TLC5947DAPR, U1 LOGIC SHIFTER, X2 SERVO, X3 POWER, X4 LOGIC

Commit message: Finished redesign of DashDial
Parts:
- removed X4: LOGIC, Rembrandt Electronics - JST XH Connectors v1-0:JST-XH-04-PIN-LONG-PAD
- added X1: LOGIC, con-wago-500:W237-4
Connections:
- net 3.3V: now also D0.A, D1.A, D10.A, D11.A, D12.A, D13.A, D14.A, D15.A, D16.A, D17.A, D18.A, D19.A, D2.A, D20.A, D21.A, D22.A, D23.A, D3.A, D4.A, D5.A, D6.A, D7.A, D8.A, D9.A, X3-1.KL; no longer X3-4.KL
- net 5V: now also X3-2.KL; no longer X3-3.KL
- net 7.4V: now also X3-3.KL; no longer X3-2.KL
- net GND: now also IC1.BLANK, X3-4.KL; no longer D0.C, D1.C, D10.C, D11.C, D12.C, D13.C, D14.C, D15.C, D16.C, D17.C, D18.C, D19.C, D2.C, D20.C, D21.C, D22.C, D23.C, D3.C, D4.C, D5.C, D6.C, D7.C, D8.C, D9.C, X3-1.KL
- net LAT: now also X1-3.KL; no longer X4-3.S
- net OUT0: now also D23.C; no longer D23.A
- net OUT1: now also D22.C; no longer D22.A
- net OUT10: now also D13.C; no longer D13.A
- net OUT11: now also D12.C; no longer D12.A
- net OUT12: now also D11.C; no longer D11.A
- net OUT13: now also D10.C; no longer D10.A
- net OUT14: now also D9.C; no longer D9.A
- net OUT15: now also D8.C; no longer D8.A
- net OUT16: now also D7.C; no longer D7.A
- net OUT17: now also D6.C; no longer D6.A
- net OUT18: now also D5.C; no longer D5.A
- net OUT19: now also D4.C; no longer D4.A
- net OUT2: now also D21.C; no longer D21.A
- net OUT20: now also D3.C; no longer D3.A
- net OUT21: now also D2.C; no longer D2.A
- net OUT22: now also D1.C; no longer D1.A
- net OUT23: now also D0.C; no longer D0.A
- net OUT3: now also D20.C; no longer D20.A
- net OUT4: now also D19.C; no longer D19.A
- net OUT5: now also D18.C; no longer D18.A
- net OUT6: now also D17.C; no longer D17.A
- net OUT7: now also D16.C; no longer D16.A
- net OUT8: now also D15.C; no longer D15.A
- net OUT9: now also D14.C; no longer D14.A
- net SCLK: now also X1-1.KL; no longer X4-1.S
- net SERVO_CTRL: now also X1-4.KL; no longer X4-4.S
- net SIN: now also X1-2.KL; no longer X4-2.S
Other:
- note added: "DashDial V2 Designer: Akash Harapanahalli"
- note removed: "DashDial V1 Designer: Akash Harapanahalli"
- moved on the sheet: C3, D0, D1, D10, D11, D12, D13, D14, D15, D16, D17, D18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

Commit message: Actually finished DashDial this time :)
Parts:
- removed X1: LOGIC, con-wago-500:W237-4
- removed X3: POWER, con-wago-500:W237-4
- added J1, J2: ESW-104-23-L-D, ESW-104-23-L-D:ESW-104-23-L-D
Connections:
- net 3.3V: now also J1.07, J2.07; no longer X3-1.KL
- net 5V: now also J1.05, J2.05; no longer X3-2.KL
- net 7.4V: now also J1.03, J2.03; no longer X3-3.KL
- net GND: now also J1.01, J2.01; no longer X3-4.KL
- net LAT: now also J1.04, J2.04; no longer X1-3.KL
- net SCLK: now also J1.08, J2.08; no longer X1-1.KL
- net SERVO_CTRL: now also J1.02, J2.02; no longer X1-4.KL
- net SIN: now also J1.06, J2.06; no longer X1-2.KL
Changed lines of the file:
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@@
 <part name="C2" library="rcl" library_urn="urn:adsk.eagle:library:334" deviceset="C-EU" device="C1206" package3d_urn="urn:adsk.eagle:package:23618/2" value="100uF"/>
 <part name="C3" library="SparkFun-Capacitors" deviceset="0.1UF" device="-0603-25V-(+80/-20%)" value="0.1uF"/>
-<part name="X3" library="con-wago-500" library_urn="urn:adsk.eagle:library:195" deviceset="W237-4" device="" package3d_urn="urn:adsk.eagle:package:10695/1" value="POWER"/>
 <part name="D0" library="SparkFun-LED" deviceset="LED" device="3MM"/>
 <part name="D1" library="SparkFun-LED" deviceset="LED" device="3MM"/>
@@
 <part name="D22" library="SparkFun-LED" deviceset="LED" device="3MM"/>
 <part name="D23" library="SparkFun-LED" deviceset="LED" device="3MM"/>
-<part name="X1" library="con-wago-500" library_urn="urn:adsk.eagle:library:195" deviceset="W237-4" device="" package3d_urn="urn:adsk.eagle:package:10695/1" value="LOGIC"/>
+<part name="J1" library="ESW-104-23-L-D" deviceset="ESW-104-23-L-D" device=""/>
+<part name="J2" library="ESW-104-23-L-D" deviceset="ESW-104-23-L-D" device=""/>
 </parts>
 <sheets>
@@
 <attribute name="VALUE" x="19.304" y="135.001" size="1.778" layer="96"/>
 </instance>
-<instance part="X3" gate="-1" x="-15.24" y="132.08" smashed="yes" rot="R180">
-<attribute name="NAME" x="-15.24" y="131.191" size="1.778" layer="95"/>
-</instance>
-<instance part="X3" gate="-2" x="-15.24" y="137.16" smashed="yes" rot="R180">
-<attribute name="NAME" x="-15.24" y="136.271" size="1.778" layer="95"/>
-</instance>
-<instance part="X3" gate="-3" x="-15.24" y="142.24" smashed="yes" rot="R180">
-<attribute name="NAME" x="-15.24" y="141.351" size="1.778" layer="95"/>
-</instance>
-<instance part="X3" gate="-4" x="-15.24" y="147.32" smashed="yes" rot="R180">
-<attribute name="VALUE" x="-12.7" y="151.003" size="1.778" layer="96" rot="R180"/>
-<attribute name="NAME" x="-15.24" y="146.431" size="1.778" layer="95"/>
-</instance>
 <instance part="D0" gate="D1" x="55.88" y="83.82" smashed="yes" rot="R270">
 <attribute name="NAME" x="51.308" y="87.249" size="1.778" layer="95" font="vector"/>
@@
 <attribute name="VALUE" x="117.348" y="28.575" size="1.778" layer="96" font="vector" align="top-left"/>
 </instance>
-<instance part="X1" gate="-1" x="-15.24" y="109.22" smashed="yes" rot="R180">
-<attribute name="NAME" x="-15.24" y="108.331" size="1.778" layer="95"/>
-</instance>
-<instance part="X1" gate="-2" x="-15.24" y="114.3" smashed="yes" rot="R180">
-<attribute name="NAME" x="-15.24" y="113.411" size="1.778" layer="95"/>
-</instance>
-<instance part="X1" gate="-3" x="-15.24" y="119.38" smashed="yes" rot="R180">
-<attribute name="NAME" x="-15.24" y="118.491" size="1.778" layer="95"/>
-</instance>
-<instance part="X1" gate="-4" x="-15.24" y="124.46" smashed="yes" rot="R180">
-<attribute name="VALUE" x="-12.7" y="128.143" size="1.778" layer="96" rot="R180"/>
-<attribute name="NAME" x="-15.24" y="123.571" size="1.778" layer="95"/>
+<instance part="J1" gate="G$1" x="-83.82" y="147.32" smashed="yes">
+<attribute name="NAME" x="-91.94" y="154.94" size="1.778" layer="95"/>
+<attribute name="VALUE" x="-91.44" y="139.7" size="1.778" layer="96"/>
+</instance>
+<instance part="J2" gate="G$1" x="-83.82" y="127" smashed="yes">
+<attribute name="NAME" x="-91.94" y="134.62" size="1.778" layer="95"/>
+<attribute name="VALUE" x="-91.44" y="119.38" size="1.778" layer="96"/>
 </instance>
 </instances>
@@
 </segment>
 <segment>
-<pinref part="X3" gate="-1" pin="KL"/>
-<wire x1="-20.32" y1="132.08" x2="-22.86" y2="132.08" width="0.1524" layer="91"/>
-<label x="-22.86" y="132.08" size="1.778" layer="95" rot="R180" xref="yes"/>
+<pinref part="J1" gate="G$1" pin="07"/>
+<wire x1="-96.52" y1="144.78" x2="-99.06" y2="144.78" width="0.1524" layer="91"/>
+<label x="-99.06" y="144.78" size="1.778" layer="95" rot="R180" xref="yes"/>
+</segment>
+<segment>
+<pinref part="J2" gate="G$1" pin="07"/>
+<wire x1="-96.52" y1="124.46" x2="-99.06" y2="124.46" width="0.1524" layer="91"/>
+<label x="-99.06" y="124.46" size="1.778" layer="95" rot="R180" xref="yes"/>
 </segment>
 </net>
@@
 </segment>
 <segment>
-<pinref part="X3" gate="-4" pin="KL"/>
-<wire x1="-20.32" y1="147.32" x2="-22.86" y2="147.32" width="0.1524" layer="91"/>
-<label x="-22.86" y="147.32" size="1.778" layer="95" rot="R180" xref="yes"/>
+<pinref part="J1" gate="G$1" pin="01"/>
+<wire x1="-96.52" y1="152.4" x2="-99.06" y2="152.4" width="0.1524" layer="91"/>
+<label x="-99.06" y="152.4" size="1.778" layer="95" rot="R180" xref="yes"/>
+</segment>
+<segment>
+<pinref part="J2" gate="G$1" pin="01"/>
+<wire x1="-96.52" y1="132.08" x2="-99.06" y2="132.08" width="0.1524" layer="91"/>
+<label x="-99.06" y="132.08" size="1.778" layer="95" rot="R180" xref="yes"/>
 </segment>
 </net>
@@
 </segment>
 <segment>
-<pinref part="X3" gate="-3" pin="KL"/>
-<wire x1="-20.32" y1="142.24" x2="-22.86" y2="142.24" width="0.1524" layer="91"/>
-<label x="-22.86" y="142.24" size="1.778" layer="95" rot="R180" xref="yes"/>
+<pinref part="J1" gate="G$1" pin="03"/>
+<wire x1="-96.52" y1="149.86" x2="-99.06" y2="149.86" width="0.1524" layer="91"/>
+<label x="-99.06" y="149.86" size="1.778" layer="95" rot="R180" xref="yes"/>
+</segment>
+<segment>
+<pinref part="J2" gate="G$1" pin="03"/>
+<wire x1="-96.52" y1="129.54" x2="-99.06" y2="129.54" width="0.1524" layer="91"/>
+<label x="-99.06" y="129.54" size="1.778" layer="95" rot="R180" xref="yes"/>
 </segment>
 </net>
@@
 </segment>
 <segment>
-<pinref part="X1" gate="-2" pin="KL"/>
-<wire x1="-20.32" y1="114.3" x2="-22.86" y2="114.3" width="0.1524" layer="91"/>
-<label x="-22.86" y="114.3" size="1.778" layer="95" rot="R180" xref="yes"/>
+<pinref part="J1" gate="G$1" pin="06"/>
+<wire x1="-71.12" y1="147.32" x2="-68.58" y2="147.32" width="0.1524" layer="91"/>
+<label x="-68.58" y="147.32" size="1.778" layer="95" xref="yes"/>
+</segment>
+<segment>
+<pinref part="J2" gate="G$1" pin="06"/>
+<wire x1="-71.12" y1="127" x2="-68.58" y2="127" width="0.1524" layer="91"/>
+<label x="-68.58" y="127" size="1.778" layer="95" xref="yes"/>
 </segment>
 </net>
@@
 </segment>
 <segment>
-<pinref part="X1" gate="-1" pin="KL"/>
-<wire x1="-20.32" y1="109.22" x2="-22.86" y2="109.22" width="0.1524" layer="91"/>
-<label x="-22.86" y="109.22" size="1.778" layer="95" rot="R180" xref="yes"/>
+<pinref part="J1" gate="G$1" pin="08"/>
+<wire x1="-71.12" y1="144.78" x2="-68.58" y2="144.78" width="0.1524" layer="91"/>
+<label x="-68.58" y="144.78" size="1.778" layer="95" xref="yes"/>
+</segment>
+<segment>
+<pinref part="J2" gate="G$1" pin="08"/>
+<wire x1="-71.12" y1="124.46" x2="-68.58" y2="124.46" width="0.1524" layer="91"/>
+<label x="-68.58" y="124.46" size="1.778" layer="95" xref="yes"/>
 </segment>
 </net>
@@
 </segment>
 <segment>
-<pinref part="X1" gate="-3" pin="KL"/>
-<wire x1="-20.32" y1="119.38" x2="-22.86" y2="119.38" width="0.1524" layer="91"/>
-<label x="-22.86" y="119.38" size="1.778" layer="95" rot="R180" xref="yes"/>
+<pinref part="J1" gate="G$1" pin="04"/>
+<wire x1="-71.12" y1="149.86" x2="-68.58" y2="149.86" width="0.1524" layer="91"/>
+<label x="-68.58" y="149.86" size="1.778" layer="95" xref="yes"/>
+</segment>
+<segment>
+<pinref part="J2" gate="G$1" pin="04"/>
+<wire x1="-71.12" y1="129.54" x2="-68.58" y2="129.54" width="0.1524" layer="91"/>
+<label x="-68.58" y="129.54" size="1.778" layer="95" xref="yes"/>
 </segment>
 </net>
@@
 </segment>
 <segment>
-<pinref part="X1" gate="-4" pin="KL"/>
-<wire x1="-20.32" y1="124.46" x2="-22.86" y2="124.46" width="0.1524" layer="91"/>
-<label x="-22.86" y="124.46" size="1.778" layer="95" rot="R180" xref="yes"/>
+<pinref part="J1" gate="G$1" pin="02"/>
+<wire x1="-71.12" y1="152.4" x2="-68.58" y2="152.4" width="0.1524" layer="91"/>
+<label x="-68.58" y="152.4" size="1.778" layer="95" xref="yes"/>
+</segment>
+<segment>
+<pinref part="J2" gate="G$1" pin="02"/>
+<wire x1="-71.12" y1="132.08" x2="-68.58" y2="132.08" width="0.1524" layer="91"/>
+<label x="-68.58" y="132.08" size="1.778" layer="95" xref="yes"/>
 </segment>
 </net>
@@
 </segment>
 <segment>
-<pinref part="X3" gate="-2" pin="KL"/>
-<wire x1="-20.32" y1="137.16" x2="-22.86" y2="137.16" width="0.1524" layer="91"/>
-<label x="-22.86" y="137.16" size="1.778" layer="95" rot="R180" xref="yes"/>
-</segment>
-</net>
+<pinref part="J1" gate="G$1" pin="05"/>
+<wire x1="-96.52" y1="147.32" x2="-99.06" y2="147.32" width="0.1524" layer="91"/>
+<label x="-99.06" y="147.32" size="1.778" layer="95" rot="R180" xref="yes"/>
+</segment>
+<segment>
+<pinref part="J2" gate="G$1" pin="05"/>
+<wire x1="-96.52" y1="127" x2="-99.06" y2="127" width="0.1524" layer="91"/>
+<label x="-99.06" y="127" size="1.778" layer="95" rot="R180" xref="yes"/>
+</segment>
+</net>
