File: Differential_Controller/Eagle Files/03-03/DiffController.brd (EAGLE design)
At the start: 67 x 58.4 mm, 29 parts, among them J1 1990083, J2 1990083, Q1 60V/32A/35mΩ, Q2 60V/32A/35mΩ, Q3 24A/20V/50mΩ, Q4 24A/20V/50mΩ, T1 BC337, T2 BC337, U1 L7805CV

Commit message: Minor changes on PCB, ready for manufacturing
Parts:
- moved C1 11.4 mm to (50.8, 53.3), turned to 270 degrees
- moved X2 8.89 mm to (59.7, 53.3)
Connections:
- net 3V3: now also R6.P$2, R8.P$2
- net 5V: no longer R6.P$2, R8.P$2
Routing:
- net 5V: track 35.2 -> 22.3 mm
- net 3V3: track 57.4 -> 66.6 mm
- net M_IN_POS: track 66.8 -> 61.3 mm
- net VBAT: track 105.6 -> 103.1 mm
- net GND: track 13.4 -> 14.3 mm, vias 0 -> 4

Commit message: Changed duplicate M_POS_IN pins on EAGLE schematic. STILL NEEDS ROUTING ON BOARD
Connections:
- net M_IN_NEG: now also R10.P$1
- net M_IN_POS: no longer R10.P$1
Routing:
- net M_IN_POS: track 61.3 -> 55.6 mm
Changed lines of the file:
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@@
 <contactref element="JP2" pad="7"/>
 <contactref element="R7" pad="P$1"/>
-<contactref element="R10" pad="P$1"/>
 <wire x1="29.40149375" y1="40.5892" x2="29.1592" y2="40.5892" width="0.2032" layer="1"/>
 <wire x1="29.1592" y1="40.5892" x2="27.94" y2="39.37" width="0.2032" layer="1"/>
@@
 <wire x1="42.03301875" y1="45.6438" x2="44.72541875" y2="48.3362" width="0.2032" layer="16"/>
 <wire x1="66.1162" y1="42.62238125" x2="64.77" y2="41.27618125" width="0.2032" layer="16"/>
-<wire x1="64.77" y1="41.27618125" x2="64.77" y2="35.56" width="0.2032" layer="16"/>
 <wire x1="44.72541875" y1="48.3362" x2="53.34" y2="48.3362" width="0.2032" layer="16"/>
 <wire x1="53.34" y1="48.3362" x2="53.7504625" y2="48.3362" width="0.2032" layer="16"/>
@@
 <contactref element="JP2" pad="6"/>
 <wire x1="27.94" y1="41.91" x2="23.749" y2="41.91" width="0.2032" layer="16"/>
+<contactref element="R10" pad="P$1"/>
+<wire x1="27.94" y1="41.91" x2="64.77" y2="35.56" width="0" layer="19" extent="1-1"/>
 </signal>
 <signal name="M_OUT_POS">
@@
 <mfgpreviewcolor name="substratecolor" color="0xFF786E46"/>
 </mfgpreviewcolors>
+<errors>
+</errors>
 </board>
 </drawing>
