File: Differential_Controller/Eagle Files/03-03/DiffController.sch (EAGLE design)
At the start: 29 parts, among them J1 1990083, J2 1990083, Q1 60V/32A/35mΩ, Q2 60V/32A/35mΩ, Q3 24A/20V/50mΩ, Q4 24A/20V/50mΩ, T1 BC337, T2 BC337, U1 L7805CV

Commit message: Minor changes on PCB, ready for manufacturing
Connections:
- net 3V3: now also R6.2, R8.2
- net 5V: no longer R6.2, R8.2
Changed lines of the file:
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@@
 <wire x1="76.2" y1="93.98" x2="93.98" y2="93.98" width="0.1524" layer="91"/>
+</segment>
+<segment>
+<pinref part="R6" gate="G$1" pin="2"/>
+<wire x1="-17.78" y1="149.86" x2="-17.78" y2="152.4" width="0.1524" layer="91"/>
+<label x="-17.78" y="152.4" size="1.778" layer="95"/>
+</segment>
+<segment>
+<pinref part="R8" gate="G$1" pin="2"/>
+<wire x1="129.54" y1="162.56" x2="129.54" y2="165.1" width="0.1524" layer="91"/>
+<label x="129.54" y="165.1" size="1.778" layer="95"/>
 </segment>
 </net>
@@
 <label x="162.56" y="83.82" size="1.778" layer="95"/>
 </segment>
-<segment>
-<pinref part="R6" gate="G$1" pin="2"/>
-<wire x1="-17.78" y1="149.86" x2="-17.78" y2="152.4" width="0.1524" layer="91"/>
-<label x="-17.78" y="152.4" size="1.778" layer="95"/>
-</segment>
-<segment>
-<pinref part="R8" gate="G$1" pin="2"/>
-<wire x1="129.54" y1="162.56" x2="129.54" y2="165.1" width="0.1524" layer="91"/>
-<label x="129.54" y="165.1" size="1.778" layer="95"/>
-</segment>
 </net>

Commit message: Changed duplicate M_POS_IN pins on EAGLE schematic. STILL NEEDS ROUTING ON BOARD
Connections:
- net M_IN_NEG: now also R10.1
- net M_IN_POS: no longer R10.1
Changed lines of the file:
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@@
 <label x="-40.64" y="132.08" size="1.778" layer="95"/>
-</segment>
-<segment>
-<pinref part="R10" gate="G$1" pin="1"/>
-<wire x1="139.7" y1="144.78" x2="144.78" y2="144.78" width="0.1524" layer="91"/>
-<label x="152.4" y="144.78" size="1.778" layer="95" rot="MR0"/>
 </segment>
 </net>
@@
 <label x="81.28" y="86.36" size="1.778" layer="95"/>
 </segment>
+<segment>
+<pinref part="R10" gate="G$1" pin="1"/>
+<wire x1="139.7" y1="144.78" x2="144.78" y2="144.78" width="0.1524" layer="91"/>
+<label x="152.4" y="144.78" size="1.778" layer="95" rot="MR0"/>
+</segment>
 </net>
