File: Auxillary_DAQ_System/2022_car/auxDaqUnitTop2022.brd (EAGLE design)
At the start: 101.6 x 83.5 mm, 23 parts

Commit message: Working on board files
Parts:
- added A10, A11, A12, A13, A14, A15, A16, A17, A18, A19, A20, A21, A22, A23, A6, A7, A8, A9: (no value), GTOR - Microfit Connector:43650-0300
- added JP4, JP5, JP6: (no value), GTOR - Connectors:1X08
- moved R2 164.5 mm to (63.5, 86.4)
- moved LED2 164.1 mm to (67.3, 86.4), turned to 270 degrees
- moved A1 157.3 mm to (15.2, 158.8), turned to 270 degrees
- moved A2 154.9 mm to (15.2, 144.8), turned to 270 degrees
- moved LED1 154.7 mm to (67.3, 82.5), turned to 270 degrees
- moved R1 154.7 mm to (63.5, 82.5)
- moved A3 152.7 mm to (15.2, 130.8), turned to 270 degrees
- moved I2C1 151.4 mm to (116.8, 149.9), turned to 90 degrees
- moved A4 150.4 mm to (15.2, 116.8), turned to 270 degrees
- moved A5 148.3 mm to (15.2, 102.9), turned to 270 degrees
- moved A0 143.3 mm to (15.2, 172.7), turned to 270 degrees
- moved I2C2 132.4 mm to (116.8, 137.2), turned to 90 degrees
- moved D3 127.8 mm to (116.8, 47.0), turned to 90 degrees
- moved D4 122.3 mm to (116.8, 62.2), turned to 90 degrees
- moved D2 120.7 mm to (116.8, 31.8), turned to 90 degrees
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Connections:
- new net ADC1: A0.P$2, JP6.1
- new net ADC10: A9.P$2, JP5.2
- new net ADC11: A10.P$2, JP5.3
- new net ADC12: A11.P$2, JP5.4
- new net ADC13: A12.P$2, JP5.5
- new net ADC14: A13.P$2, JP5.6
- new net ADC15: A14.P$2, JP5.7
- new net ADC16: A15.P$2, JP5.8
- new net ADC17: A16.P$2, JP4.1
- new net ADC18: A17.P$2, JP4.2
- new net ADC19: A18.P$2, JP4.3
- new net ADC2: A1.P$2, JP6.2
- new net ADC20: A19.P$2, JP4.4
- new net ADC21: A20.P$2, JP4.5
- new net ADC22: A21.P$2, JP4.6
- new net ADC23: A22.P$2, JP4.7
- new net ADC24: A23.P$2, JP4.8
- new net ADC3: A2.P$2, JP6.3
- new net ADC4: A3.P$2, JP6.4
- new net ADC5: A4.P$2, JP6.5
- new net ADC6: A5.P$2, JP6.6
- new net ADC7: A6.P$2, JP6.7
- new net ADC8: A7.P$2, JP6.8
- new net ADC9: A8.P$2, JP5.1
- net +3V3: no longer A0.P$1, A1.P$1, A2.P$1, A3.P$1, A4.P$1, A5.P$1
- net +5V: now also A0.P$1, A1.P$1, A10.P$1, A11.P$1, A12.P$1, A13.P$1, A14.P$1, A15.P$1, A16.P$1, A17.P$1, A18.P$1, A19.P$1, A2.P$1, A20.P$1, A21.P$1, A22.P$1, A23.P$1, A3.P$1, A4.P$1, A5.P$1, A6.P$1, A7.P$1, A8.P$1, A9.P$1
- net 30: no longer R1.1
- net 33: now also R1.1
- net 36: no longer CS=3.P$2
- net 9: now also CS=3.P$2
- net A0: no longer A0.P$2
- net A1: no longer A1.P$2
- net A2: no longer A2.P$2
- net A3: no longer A3.P$2
- net A6: no longer A4.P$2
- net A7: no longer A5.P$2
- net GND: now also A10.P$3, A11.P$3, A12.P$3, A13.P$3, A14.P$3, A15.P$3, A16.P$3, A17.P$3, A18.P$3, A19.P$3, A20.P$3, A21.P$3, A22.P$3, A23.P$3, A6.P$3, A7.P$3, A8.P$3, A9.P$3
Routing:
- net SCL: track 0.00 -> 169.0 mm
- net SDA: track 0.00 -> 165.9 mm
- net SCK: track 0.00 -> 138.7 mm, vias 0 -> 1
- net 9: track 0.00 -> 112.7 mm
- net MISO: track 0.00 -> 106.6 mm
- net MOSI: track 0.00 -> 103.5 mm
- net 8: track 0.00 -> 94.7 mm
- net ADC24: track 0.00 -> 87.9 mm
- net 7: track 0.00 -> 82.0 mm
- net ADC23: track 0.00 -> 71.0 mm
- net 6: track 0.00 -> 69.3 mm
- net ADC22: track 0.00 -> 59.5 mm
- net 5: track 0.00 -> 57.8 mm
- net ADC21: track 0.00 -> 48.7 mm
- net ADC13: track 0.00 -> 46.8 mm
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- added copper zone on layer 16, net +3V3
- added copper zone on layer 16, net +5V
- added copper zone on layer 1, net GND
Other:
- board size 101.6 x 83.5 mm -> 121.9 x 193 mm
- board text added: "2"
- board text added: "2022 AuxDAQ Top rev1 Peter Chu"
- board text added: "3"
- board text added: "3.3v"
- board text added: "4"
- board text added: "5"
- board text added: "6"
- board text added: "7"
- board text added: "ADC1-12"
- board text added: "ADC13-24"
- board text added: "CS=8"
- board text added: "CS=9"
- board text added: "DIGITAL"
- board text added: "Debug Pin 30"
- board text added: "I2C"
- board text added: "SPI"
