File: Auxillary_DAQ_System/2022_car/auxDaqUnitTop2022.sch (EAGLE design)
At the start: 23 parts

Commit message: Working on board files
Parts:
- added A10, A11, A12, A13, A14, A15, A16, A17, A18, A19, A20, A21, A22, A23, A6, A7, A8, A9: (no value), GTOR - Microfit Connector:HEADER_POS3_43650-0300
- added JP4, JP5, JP6: (no value), GTOR - Connectors:PINHD-1X8
Connections:
- new net ADC1: A0.2, JP6.1
- new net ADC10: A9.2, JP5.2
- new net ADC11: A10.2, JP5.3
- new net ADC12: A11.2, JP5.4
- new net ADC13: A12.2, JP5.5
- new net ADC14: A13.2, JP5.6
- new net ADC15: A14.2, JP5.7
- new net ADC16: A15.2, JP5.8
- new net ADC17: A16.2, JP4.1
- new net ADC18: A17.2, JP4.2
- new net ADC19: A18.2, JP4.3
- new net ADC2: A1.2, JP6.2
- new net ADC20: A19.2, JP4.4
- new net ADC21: A20.2, JP4.5
- new net ADC22: A21.2, JP4.6
- new net ADC23: A22.2, JP4.7
- new net ADC24: A23.2, JP4.8
- new net ADC3: A2.2, JP6.3
- new net ADC4: A3.2, JP6.4
- new net ADC5: A4.2, JP6.5
- new net ADC6: A5.2, JP6.6
- new net ADC7: A6.2, JP6.7
- new net ADC8: A7.2, JP6.8
- new net ADC9: A8.2, JP5.1
- net +3V3: no longer A0.1, A1.1, A2.1, A3.1, A4.1, A5.1
- net +5V: now also A0.1, A1.1, A10.1, A11.1, A12.1, A13.1, A14.1, A15.1, A16.1, A17.1, A18.1, A19.1, A2.1, A20.1, A21.1, A22.1, A23.1, A3.1, A4.1, A5.1, A6.1, A7.1, A8.1, A9.1
- net 30: no longer R1.1
- net 33: now also R1.1
- net 36: no longer CS=3.2
- net 9: now also CS=3.2
- net A0: no longer A0.2
- net A1: no longer A1.2
- net A2: no longer A2.2
- net A3: no longer A3.2
- net A6: no longer A4.2
- net A7: no longer A5.2
- net GND: now also A10.3, A11.3, A12.3, A13.3, A14.3, A15.3, A16.3, A17.3, A18.3, A19.3, A20.3, A21.3, A22.3, A23.3, A6.3, A7.3, A8.3, A9.3
Other:
- moved on the sheet: A0, A1, A2, A3, A4, A5, D1, D2, D3, D4, D5, D6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
