File: Auxillary_DAQ_System/2022_car/auxDaqUnitTopDigital2022.brd (EAGLE design)
At the start: 38.1 x 156.2 mm, 26 parts

Commit message: Minor DRC fixes and trace thickening
Parts:
- removed JP3: (no value), GTOR - Connectors:1X03
- added JP1: (no value), GTOR - Connectors:1X02
Connections:
- removed net +5V: JP3.3
- net +3V3: now also JP1.2; no longer JP3.2
- net GND: now also JP1.1; no longer JP3.1
Changed lines of the file:
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@@
 </autorouter>
 <elements>
-<element name="JP3" library="GTOR - Connectors" package="1X03" package3d_urn="urn:adsk.eagle:package:22458/2" value="" x="102.87" y="49.53" smashed="yes" rot="R90">
-<attribute name="NAME" x="101.0412" y="45.6438" size="1.27" layer="25" ratio="10" rot="R90"/>
-<attribute name="POPULARITY" value="92" x="102.87" y="49.53" size="1.778" layer="27" rot="R90" display="off"/>
-<attribute name="VALUE" x="106.045" y="45.72" size="1.27" layer="27" rot="R90"/>
-</element>
 <element name="CS=10" library="GTOR - Microfit Connector" package="43045-0600" value="" x="116.84" y="135.89" smashed="yes" rot="R90"/>
 <element name="D1" library="GTOR - Microfit Connector" package="43650-0300" value="" x="116.84" y="52.07" smashed="yes" rot="R90"/>
@@
 <attribute name="POPULARITY" value="1" x="102.87" y="110.49" size="1.778" layer="27" rot="R90" display="off"/>
 <attribute name="VALUE" x="106.045" y="82.55" size="1.27" layer="27" rot="R90"/>
+</element>
+<element name="JP1" library="GTOR - Connectors" package="1X02" package3d_urn="urn:adsk.eagle:package:22435/2" value="" x="102.87" y="49.53" smashed="yes" rot="R90">
+<attribute name="NAME" x="101.0412" y="46.9138" size="1.27" layer="25" ratio="10" rot="R90"/>
+<attribute name="POPULARITY" value="98" x="102.87" y="49.53" size="1.778" layer="27" rot="R90" display="off"/>
+<attribute name="VALUE" x="106.045" y="46.99" size="1.27" layer="27" rot="R90"/>
 </element>
 </elements>
@@
 </signal>
 <signal name="GND">
-<contactref element="JP3" pad="1"/>
 <contactref element="D1" pad="P$3"/>
 <contactref element="I2C1" pad="P$4"/>
@@
 <vertex x="74.93" y="204.47"/>
 </polygon>
-</signal>
-<signal name="+5V">
-<contactref element="JP3" pad="3"/>
+<contactref element="JP1" pad="1"/>
 </signal>
 <signal name="+3V3">
-<contactref element="JP3" pad="2"/>
 <contactref element="CS=10" pad="P$1"/>
 <contactref element="I2C1" pad="P$1"/>
@@
 <wire x1="102.02" y1="55.88" x2="100.33" y2="55.88" width="0.1524" layer="1"/>
 <via x="100.33" y="55.88" extent="1-16" drill="0.35"/>
+<contactref element="JP1" pad="2"/>
 </signal>
 <signal name="2">
