File: Dashboard/2021 Dashboard/DashHub.brd (EAGLE design)
At the start: 86.4 x 66 mm, 32 parts, among them J1 LEFT, J2 RIGHT, U1 ALLEGRO_MICROSYSTEMS_ACS722LL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, U2 XBEE_PRO_S3B

Commit message: Added OLED
Connections:
- removed net LAT_D: JP3.12, U$1.15/A1
- removed net SIN_D: JP3.13, U$1.14/A0
- new net SCL: JP3.12, U$1.15/A1, U$2.SCL
- new net SDA: JP3.13, U$1.14/A0, U$2.SDA
Routing:
- net SIN_D: track 3.81 -> 0.00 mm
- net SDA: track 0.00 -> 3.81 mm
- net SCL: track 0.00 -> 3.81 mm
- net LAT_D: track 3.81 -> 0.00 mm
Changed lines of the file:
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@@
 <wire x1="-17.4498" y1="-7.6962" x2="-7.692275" y2="-1.5748" width="0" layer="19" extent="16-16"/>
 </signal>
-<signal name="LAT_D">
+<signal name="SCL">
 <contactref element="U$1" pad="15/A1"/>
 <contactref element="JP3" pad="12"/>
 <wire x1="-11.43" y1="-22.86" x2="-7.62" y2="-22.86" width="0.1524" layer="1"/>
+<contactref element="U$2" pad="SCL"/>
+<wire x1="1.27" y1="30.353" x2="-7.62" y2="-22.86" width="0" layer="19" extent="1-1"/>
 </signal>
 <signal name="SCLK_D">
@@
 <wire x1="-11.43" y1="-27.94" x2="-7.62" y2="-27.94" width="0.1524" layer="1"/>
 </signal>
-<signal name="SIN_D">
+<signal name="SDA">
 <contactref element="U$1" pad="14/A0"/>
 <contactref element="JP3" pad="13"/>
 <wire x1="-11.43" y1="-25.4" x2="-7.62" y2="-25.4" width="0.1524" layer="1"/>
+<contactref element="U$2" pad="SDA"/>
+<wire x1="3.81" y1="30.353" x2="-7.62" y2="-25.4" width="0" layer="19" extent="1-1"/>
 </signal>
 <signal name="ENGINE_RPM">
