File: Dashboard/2021 Dashboard/DashHub.sch (EAGLE design)
At the start: 26 parts, among them J1 LEFT, J2 RIGHT, U1 ALLEGRO_MICROSYSTEMS_ACS722LL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

Commit message: Linear Regulator
Parts:
- removed U$3: DC-DC-STEP-DOWN-MP1584, diy-modules:DC-DC-STEP-DOWN-MP1584
- added C3: 10uF, GTOR - Passive Components:CAP_SMDC1206
- added C5, C6: 47uF, GTOR - Passive Components:CAP_SMDC1206
- added U$6: TPSM84205EAB, GTOR - Active Components:TPSM84205EAB
Connections:
- removed net 3.3V_BUCK: J1.08, J2.08, U$3.OUT+.1, U$3.OUT+.2
- new net 3.3V_REG: C5.1, C6.1, J1.08, J2.08, U$6.VOUT
- net 7.4V: now also C3.2, U$6.VIN; no longer U$3.IN+.1, U$3.IN+.2
- net GND: now also U$6.GND; no longer U$3.IN-.1, U$3.IN-.2, U$3.OUT-.1, U$3.OUT-.2
Changed lines of the file:
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@@
 <part name="JP5" library="pinhead" library_urn="urn:adsk.eagle:library:325" deviceset="PINHD-2X5" device="" package3d_urn="urn:adsk.eagle:package:22470/2"/>
 <part name="U$2" library="diy-modules" deviceset="DC-DC-STEP-DOWN-MP1584" device=""/>
-<part name="U$3" library="diy-modules" deviceset="DC-DC-STEP-DOWN-MP1584" device=""/>
 <part name="U$4" library="GTOR - Connectors" deviceset="48CKTRASCMCHEADER" device=""/>
 <part name="U$5" library="GTOR - Breakout Boards" deviceset="DIYMALL_6M_GPS_BREAKOUT" device=""/>
 <part name="+3V1" library="GTOR - Documation Frame" deviceset="+3V3" device=""/>
+<part name="U$6" library="GTOR - Active Components" deviceset="TPSM84205EAB" device=""/>
+<part name="C3" library="GTOR - Passive Components" deviceset="CAP_SMD" device="C1206" package3d_urn="urn:adsk.eagle:package:23618/2" value="10uF"/>
+<part name="C5" library="GTOR - Passive Components" deviceset="CAP_SMD" device="C1206" package3d_urn="urn:adsk.eagle:package:23618/2" value="47uF"/>
+<part name="C6" library="GTOR - Passive Components" deviceset="CAP_SMD" device="C1206" package3d_urn="urn:adsk.eagle:package:23618/2" value="47uF"/>
 </parts>
 <sheets>
@@
 <attribute name="VALUE" x="27.94" y="0" size="1.778" layer="96"/>
 </instance>
-<instance part="U$3" gate="G$1" x="40.64" y="-43.18" smashed="yes">
-<attribute name="NAME" x="27.94" y="-27.94" size="1.778" layer="95"/>
-<attribute name="VALUE" x="27.94" y="-30.48" size="1.778" layer="96"/>
-</instance>
 <instance part="U$4" gate="G$1" x="27.94" y="27.94" smashed="yes">
 <attribute name="NAME" x="-3.81" y="33.655" size="1.778" layer="95"/>
@@
 <instance part="+3V1" gate="G$1" x="109.22" y="129.54" smashed="yes">
 <attribute name="VALUE" x="106.68" y="124.46" size="1.778" layer="96" rot="R90"/>
+</instance>
+<instance part="U$6" gate="G$1" x="25.4" y="-27.94" smashed="yes">
+<attribute name="NAME" x="27.94" y="-30.48" size="2.54" layer="95" align="top-left"/>
+</instance>
+<instance part="C3" gate="G$1" x="20.32" y="-45.72" smashed="yes" rot="R180">
+<attribute name="NAME" x="18.796" y="-46.101" size="1.778" layer="95" rot="R180"/>
+<attribute name="VALUE" x="18.796" y="-41.021" size="1.778" layer="96" rot="R180"/>
+</instance>
+<instance part="C5" gate="G$1" x="68.58" y="-43.18" smashed="yes">
+<attribute name="NAME" x="70.104" y="-42.799" size="1.778" layer="95"/>
+<attribute name="VALUE" x="70.104" y="-47.879" size="1.778" layer="96"/>
+</instance>
+<instance part="C6" gate="G$1" x="78.74" y="-43.18" smashed="yes">
+<attribute name="NAME" x="80.264" y="-42.799" size="1.778" layer="95"/>
+<attribute name="VALUE" x="80.264" y="-47.879" size="1.778" layer="96"/>
 </instance>
 </instances>
@@
 </segment>
 <segment>
-<pinref part="U$3" gate="G$1" pin="IN-.1"/>
-<pinref part="U$3" gate="G$1" pin="IN-.2"/>
-<wire x1="22.86" y1="-38.1" x2="22.86" y2="-40.64" width="0.1524" layer="91"/>
-<wire x1="22.86" y1="-40.64" x2="20.32" y2="-40.64" width="0.1524" layer="91"/>
-<junction x="22.86" y="-40.64"/>
-<label x="20.32" y="-40.64" size="1.778" layer="95" rot="R180" xref="yes"/>
-</segment>
-<segment>
-<pinref part="U$3" gate="G$1" pin="OUT-.1"/>
-<pinref part="U$3" gate="G$1" pin="OUT-.2"/>
-<wire x1="58.42" y1="-38.1" x2="58.42" y2="-40.64" width="0.1524" layer="91"/>
-<wire x1="58.42" y1="-40.64" x2="60.96" y2="-40.64" width="0.1524" layer="91"/>
-<junction x="58.42" y="-40.64"/>
-<label x="60.96" y="-40.64" size="1.778" layer="95" xref="yes"/>
-</segment>
-<segment>
 <label x="51.562" y="38.1" size="1.778" layer="95" xref="yes"/>
 <pinref part="U$4" gate="G$1" pin="2B"/>
@@
 <wire x1="116.84" y1="116.84" x2="109.22" y2="116.84" width="0.1524" layer="91"/>
 <pinref part="U$5" gate="G$1" pin="GND"/>
+</segment>
+<segment>
+<wire x1="55.88" y1="-40.64" x2="58.42" y2="-40.64" width="0.1524" layer="91"/>
+<label x="58.42" y="-40.64" size="1.778" layer="95" xref="yes"/>
+<pinref part="U$6" gate="G$1" pin="GND"/>
 </segment>
 </net>
@@
 </segment>
 <segment>
-<pinref part="U$3" gate="G$1" pin="IN+.1"/>
-<pinref part="U$3" gate="G$1" pin="IN+.2"/>
-<wire x1="22.86" y1="-45.72" x2="22.86" y2="-48.26" width="0.1524" layer="91"/>
-<wire x1="22.86" y1="-48.26" x2="20.32" y2="-48.26" width="0.1524" layer="91"/>
-<junction x="22.86" y="-48.26"/>
-<label x="20.32" y="-48.26" size="1.778" layer="95" rot="R180" xref="yes"/>
+<wire x1="22.86" y1="-35.56" x2="20.32" y2="-35.56" width="0.1524" layer="91"/>
+<label x="15.24" y="-35.56" size="1.778" layer="95" rot="R180" xref="yes"/>
+<pinref part="U$6" gate="G$1" pin="VIN"/>
+<wire x1="20.32" y1="-35.56" x2="15.24" y2="-35.56" width="0.1524" layer="91"/>
+<wire x1="20.32" y1="-35.56" x2="20.32" y2="-40.64" width="0.1524" layer="91"/>
+<junction x="20.32" y="-35.56"/>
+<pinref part="C3" gate="G$1" pin="2"/>
 </segment>
 </net>
@@
 </segment>
 </net>
-<net name="3.3V_BUCK" class="0">
+<net name="3.3V_REG" class="0">
 <segment>
 <pinref part="J1" gate="G$1" pin="08"/>
@@
 </segment>
 <segment>
-<pinref part="U$3" gate="G$1" pin="OUT+.1"/>
-<pinref part="U$3" gate="G$1" pin="OUT+.2"/>
-<wire x1="58.42" y1="-45.72" x2="58.42" y2="-48.26" width="0.1524" layer="91"/>
-<wire x1="58.42" y1="-48.26" x2="60.96" y2="-48.26" width="0.1524" layer="91"/>
-<junction x="58.42" y="-48.26"/>
-<label x="60.96" y="-48.26" size="1.778" layer="95" xref="yes"/>
+<wire x1="55.88" y1="-35.56" x2="68.58" y2="-35.56" width="0.1524" layer="91"/>
+<label x="83.82" y="-35.56" size="1.778" layer="95" xref="yes"/>
+<pinref part="U$6" gate="G$1" pin="VOUT"/>
+<wire x1="68.58" y1="-35.56" x2="78.74" y2="-35.56" width="0.1524" layer="91"/>
+<wire x1="78.74" y1="-35.56" x2="83.82" y2="-35.56" width="0.1524" layer="91"/>
+<wire x1="68.58" y1="-35.56" x2="68.58" y2="-40.64" width="0.1524" layer="91"/>
+<junction x="68.58" y="-35.56"/>
+<wire x1="78.74" y1="-40.64" x2="78.74" y2="-35.56" width="0.1524" layer="91"/>
+<junction x="78.74" y="-35.56"/>
+<pinref part="C5" gate="G$1" pin="1"/>
+<pinref part="C6" gate="G$1" pin="1"/>
 </segment>
 </net>
@@
 packages will not be understood (or retained) with this version.
 </note>
+<note version="8.4" severity="warning">
+Since Version 8.4, EAGLE supports properties for SPICE simulation.
+Probes in schematics and SPICE mapping objects found in parts and library devices
+will not be understood with this version. Update EAGLE to the latest version
+for full support of SPICE simulation.
+</note>
 </compatibility>

Commit message: Added new linear regulator and XBee silkscreen to dashhub
Parts:
- removed JP1: (no value), SparkFun-RF:XBEE
- removed U$2: DC-DC-STEP-DOWN-MP1584, diy-modules:DC-DC-STEP-DOWN-MP1584
- added C2: 4.7uF, GTOR - Passive Components:CAP_SMDC0603
- added C4: 1uF, GTOR - Passive Components:CAP_SMDC1206
- added U$3: REG_5V_LDL1117S50R, GTOR - Active Components:REG_5V_LDL1117S50R
- added U2: XBEE_PRO_S3B, GTOR - Microcontroller:XBEE_PRO_S3B
Connections:
- net 3.3V_TEENSY: now also U2.VCC; no longer JP1.VDD
- net 5V: now also C2.1, U$3.OUT; no longer U$2.OUT+.1, U$2.OUT+.2
- net 7.4V: now also C4.1, U$3.IN; no longer U$2.IN+.1, U$2.IN+.2
- net GND: now also C2.2, C4.2, U$3.GND, U2.GND; no longer JP1.GND, U$2.IN-.1, U$2.IN-.2, U$2.OUT-.1, U$2.OUT-.2
- net XBEE_RX: now also U2.DOUT/DIO13; no longer JP1.DOUT
- net XBEE_TX: now also U2.DIN/NCONFIG/DIO14; no longer JP1.DIN

Commit message: Added gps to dashhub
Parts:
- added U$2: OLED_SSD1306, GTOR - Breakout Boards:OLED_SSD1306
Connections:
- net 5V: now also U$2.VCC
- net GND: now also U$2.GND
Changed lines of the file:
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@@
 <part name="C4" library="GTOR - Passive Components" deviceset="CAP_SMD" device="C1206" package3d_urn="urn:adsk.eagle:package:23618/2" value="1uF"/>
 <part name="U2" library="GTOR - Microcontroller" deviceset="XBEE_PRO_S3B" device=""/>
+<part name="U$2" library="GTOR - Breakout Boards" deviceset="OLED_SSD1306" device=""/>
 </parts>
 <sheets>
@@
 <attribute name="VALUE" x="134.5709" y="-40.6946" size="1.27271875" layer="96"/>
 </instance>
+<instance part="U$2" gate="G$1" x="177.8" y="116.84" smashed="yes"/>
 </instances>
 <busses>
@@
 <label x="187.96" y="-35.56" size="1.778" layer="95" xref="yes"/>
 </segment>
+<segment>
+<wire x1="170.18" y1="111.76" x2="167.64" y2="111.76" width="0.1524" layer="91"/>
+<pinref part="U$2" gate="G$1" pin="GND"/>
+<label x="167.64" y="111.76" size="1.778" layer="95" rot="R180" xref="yes"/>
+</segment>
 </net>
 <net name="LAT_L" class="0">
@@
 <label x="50.8" y="-5.08" size="1.778" layer="95" xref="yes"/>
 </segment>
-</net>
+<segment>
+<wire x1="167.64" y1="114.3" x2="170.18" y2="114.3" width="0.1524" layer="91"/>
+<pinref part="U$2" gate="G$1" pin="VCC"/>
+<label x="167.64" y="114.3" size="1.778" layer="95" rot="R180" xref="yes"/>
+</segment>
+</net>

Commit message: Added OLED
Connections:
- removed net LAT_D: JP3.12, U$1.15/A1/RX3
- removed net SIN_D: JP3.13, U$1.14/A0/TX3
- new net SCL: JP3.12, U$1.15/A1/RX3, U$2.SCL
- new net SDA: JP3.13, U$1.14/A0/TX3, U$2.SDA
Changed lines of the file:
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@@
 </segment>
 </net>
-<net name="LAT_D" class="0">
+<net name="SCL" class="0">
 <segment>
 <pinref part="U$1" gate="G$1" pin="15/A1/RX3"/>
 <wire x1="175.26" y1="53.34" x2="180.34" y2="53.34" width="0.1524" layer="91"/>
-<label x="187.96" y="53.34" size="1.778" layer="95" xref="yes"/>
 <pinref part="JP3" gate="A" pin="12"/>
 <wire x1="180.34" y1="53.34" x2="187.96" y2="53.34" width="0.1524" layer="91"/>
 <junction x="180.34" y="53.34"/>
+<label x="187.96" y="53.34" size="1.778" layer="95" xref="yes"/>
+</segment>
+<segment>
+<wire x1="170.18" y1="119.38" x2="162.56" y2="119.38" width="0.1524" layer="91"/>
+<label x="162.56" y="119.38" size="1.778" layer="95" rot="R180" xref="yes"/>
+<pinref part="U$2" gate="G$1" pin="SCL"/>
 </segment>
 </net>
@@
 <pinref part="U$1" gate="G$1" pin="13/SCK"/>
 <wire x1="175.26" y1="48.26" x2="180.34" y2="48.26" width="0.1524" layer="91"/>
-<label x="187.96" y="48.26" size="1.778" layer="95" xref="yes"/>
 <pinref part="JP3" gate="A" pin="14"/>
-<wire x1="180.34" y1="48.26" x2="187.96" y2="48.26" width="0.1524" layer="91"/>
-<junction x="180.34" y="48.26"/>
 </segment>
 </net>
-<net name="SIN_D" class="0">
+<net name="SDA" class="0">
 <segment>
 <pinref part="U$1" gate="G$1" pin="14/A0/TX3"/>
 <wire x1="175.26" y1="50.8" x2="180.34" y2="50.8" width="0.1524" layer="91"/>
-<label x="187.96" y="50.8" size="1.778" layer="95" xref="yes"/>
 <pinref part="JP3" gate="A" pin="13"/>
 <wire x1="180.34" y1="50.8" x2="187.96" y2="50.8" width="0.1524" layer="91"/>
 <junction x="180.34" y="50.8"/>
+<label x="187.96" y="50.8" size="1.778" layer="95" xref="yes"/>
+</segment>
+<segment>
+<wire x1="170.18" y1="121.92" x2="162.56" y2="121.92" width="0.1524" layer="91"/>
+<label x="162.56" y="121.92" size="1.778" layer="95" rot="R180" xref="yes"/>
+<pinref part="U$2" gate="G$1" pin="SDA"/>
 </segment>
 </net>

Commit message: Making space for the OLED
Connections:
- net 5V: no longer J1.06, J2.06
- net GND: now also C3.1, C5.2, C6.2
Changed lines of the file:
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@@
 <label x="167.64" y="111.76" size="1.778" layer="95" rot="R180" xref="yes"/>
+</segment>
+<segment>
+<wire x1="20.32" y1="-48.26" x2="20.32" y2="-50.8" width="0.1524" layer="91"/>
+<label x="20.32" y="-50.8" size="1.778" layer="95" rot="R270" xref="yes"/>
+<pinref part="C3" gate="G$1" pin="1"/>
+</segment>
+<segment>
+<wire x1="68.58" y1="-48.26" x2="68.58" y2="-50.8" width="0.1524" layer="91"/>
+<label x="68.58" y="-50.8" size="1.778" layer="95" rot="R270" xref="yes"/>
+<pinref part="C5" gate="G$1" pin="2"/>
+</segment>
+<segment>
+<wire x1="78.74" y1="-48.26" x2="78.74" y2="-50.8" width="0.1524" layer="91"/>
+<label x="78.74" y="-50.8" size="1.778" layer="95" rot="R270" xref="yes"/>
+<pinref part="C6" gate="G$1" pin="2"/>
 </segment>
 </net>
@@
 </segment>
 <segment>
-<pinref part="J1" gate="G$1" pin="06"/>
-<wire x1="58.42" y1="76.2" x2="60.96" y2="76.2" width="0.1524" layer="91"/>
-<label x="60.96" y="76.2" size="1.778" layer="95" xref="yes"/>
-</segment>
-<segment>
 <wire x1="53.34" y1="30.48" x2="53.34" y2="43.18" width="0.1524" layer="91"/>
 <label x="53.34" y="43.18" size="1.778" layer="95" xref="yes"/>
@@
 </segment>
 <segment>
-<wire x1="58.42" y1="55.88" x2="60.96" y2="55.88" width="0.1524" layer="91"/>
-<label x="60.96" y="55.88" size="1.778" layer="95" xref="yes"/>
-<pinref part="J2" gate="G$1" pin="06"/>
-</segment>
-<segment>
