File: Misc_Projects/Comms_Testing/Eagle Files/CommsTestBoard/CommsTestBoard.brd (EAGLE design)
At the start: 76.2 x 100 mm, 12 parts, among them J1 1985205, J2 1985205

Commit message: Fixing OLED for testing board
Parts:
- moved U$4 21.6 mm to (29.2, 92.7), turned to 270 degrees
Routing:
- net SCL: track 37.6 -> 63.3 mm
- net SDA: track 37.2 -> 58.6 mm
- net 3V3: track 163.0 -> 181.9 mm
Changed lines of the file:
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@@
 <autorouter>
 <pass name="Default">
-<param name="RoutingGrid" value="50mil"/>
+<param name="RoutingGrid" value="6.25mil"/>
 <param name="AutoGrid" value="1"/>
 <param name="Efforts" value="1"/>
 <param name="TopRouterVariant" value="1"/>
 <param name="tpViaShape" value="round"/>
-<param name="PrefDir.1" value="a"/>
+<param name="PrefDir.1" value="*"/>
 <param name="PrefDir.2" value="0"/>
 <param name="PrefDir.3" value="0"/>
@@
 <param name="PrefDir.14" value="0"/>
 <param name="PrefDir.15" value="0"/>
-<param name="PrefDir.16" value="a"/>
+<param name="PrefDir.16" value="*"/>
 <param name="cfVia" value="8"/>
 <param name="cfNonPref" value="5"/>
@@
 <attribute name="NAME" x="57.96" y="70.36" size="1.27" layer="25"/>
 </element>
-<element name="U$4" library="GTOR - Breakout Boards" package="OLED_SSD1306" value="OLED_SSD1306" x="29.21" y="71.12" smashed="yes" rot="R90">
-<attribute name="NAME" x="16.2988" y="75.0862" size="1.27" layer="25" ratio="10" rot="R270"/>
+<element name="U$4" library="GTOR - Breakout Boards" package="OLED_SSD1306" value="OLED_SSD1306" x="29.21" y="92.71" smashed="yes" rot="R270">
+<attribute name="NAME" x="42.1212" y="88.7438" size="1.27" layer="25" ratio="10" rot="R90"/>
 </element>
 </elements>
@@
 <contactref element="J1" pad="3"/>
 <contactref element="J2" pad="3"/>
+<wire x1="30.48" y1="54.61" x2="49.96" y2="70.05" width="0" layer="19" extent="1-1"/>
+<wire x1="6.32" y1="51.63" x2="30.48" y2="54.61" width="0" layer="19" extent="1-1"/>
+<wire x1="5.08" y1="40.56" x2="6.32" y2="51.63" width="0" layer="19" extent="1-1"/>
+<wire x1="6.32" y1="12.26" x2="5.08" y2="40.56" width="0" layer="19" extent="1-1"/>
+<wire x1="30.48" y1="19.05" x2="6.32" y2="12.26" width="0" layer="19" extent="1-1"/>
+<wire x1="5.08" y1="81.2" x2="6.32" y2="51.63" width="0" layer="19" extent="1-1"/>
+<wire x1="25.4" y1="92.71" x2="5.08" y2="81.2" width="0" layer="19" extent="1-1"/>
+<wire x1="69.85" y1="45.72" x2="49.96" y2="70.05" width="0" layer="19" extent="1-1"/>
+<wire x1="69.85" y1="11.43" x2="69.85" y2="45.72" width="0" layer="19" extent="1-1"/>
 </signal>
 <signal name="3V3">
@@
 <wire x1="3.175" y1="35.56" x2="3.175" y2="57.15" width="0.1524" layer="1"/>
 <wire x1="5.715" y1="58.42" x2="6.32" y2="58.63" width="0.1524" layer="1"/>
-<wire x1="34.925" y1="73.025" x2="49.53" y2="87.63" width="0.1524" layer="1"/>
-<wire x1="32.385" y1="73.025" x2="34.925" y2="73.025" width="0.1524" layer="1"/>
-<wire x1="30.48" y1="71.12" x2="32.385" y2="73.025" width="0.1524" layer="1"/>
 <wire x1="49.53" y1="87.63" x2="49.96" y2="88.05" width="0.1524" layer="1"/>
 <wire x1="53.34" y1="59.69" x2="67.31" y2="45.72" width="0.1524" layer="1"/>
 <wire x1="53.34" y1="86.36" x2="53.34" y2="59.69" width="0.1524" layer="1"/>
 <wire x1="50.165" y1="87.63" x2="52.07" y2="87.63" width="0.1524" layer="1"/>
-<wire x1="50.165" y1="87.63" x2="49.96" y2="88.05" width="0.1524" layer="1"/>
-<wire x1="6.35" y1="73.025" x2="5.08" y2="71.755" width="0.1524" layer="1"/>
-<wire x1="32.385" y1="73.025" x2="6.35" y2="73.025" width="0.1524" layer="1"/>
+<wire x1="50.165" y1="87.63" x2="50.042825" y2="87.880309375" width="0.1524" layer="1"/>
+<wire x1="50.042825" y1="87.880309375" x2="49.96" y2="88.05" width="0.1524" layer="1"/>
 <wire x1="5.08" y1="71.755" x2="5.08" y2="71.2" width="0.1524" layer="1"/>
 <wire x1="52.07" y1="87.63" x2="53.34" y2="86.36" width="0.1524" layer="1"/>
 <wire x1="3.175" y1="57.15" x2="4.445" y2="58.42" width="0.1524" layer="1"/>
 <wire x1="4.445" y1="58.42" x2="5.715" y2="58.42" width="0.1524" layer="1"/>
+<wire x1="5.08" y1="71.755" x2="12.7" y2="79.375" width="0.1524" layer="1"/>
+<wire x1="12.7" y1="79.375" x2="12.7" y2="95.25" width="0.1524" layer="1"/>
+<wire x1="12.7" y1="95.25" x2="26.67" y2="95.25" width="0.1524" layer="1"/>
+<wire x1="26.67" y1="95.25" x2="46.99" y2="95.25" width="0.1524" layer="1"/>
+<wire x1="46.99" y1="95.25" x2="50.042825" y2="92.197175" width="0.1524" layer="1"/>
+<wire x1="50.042825" y1="92.197175" x2="50.042825" y2="87.880309375" width="0.1524" layer="1"/>
+<wire x1="26.67" y1="95.25" x2="27.94" y2="93.98" width="0.1524" layer="1"/>
+<wire x1="27.94" y1="93.98" x2="27.94" y2="92.71" width="0.1524" layer="1"/>
 </signal>
 <signal name="T3">
@@
 <contactref element="U$4" pad="SDA"/>
 <contactref element="U$2" pad="18/A4/SDA"/>
-<wire x1="28.575" y1="69.215" x2="52.07" y2="45.72" width="0.1524" layer="1"/>
-<wire x1="27.305" y1="69.215" x2="28.575" y2="69.215" width="0.1524" layer="1"/>
-<wire x1="25.4" y1="71.12" x2="27.305" y2="69.215" width="0.1524" layer="1"/>
+<wire x1="52.07" y1="45.72" x2="28.575" y2="69.215" width="0.1524" layer="1"/>
+<wire x1="28.575" y1="69.215" x2="28.575" y2="84.455" width="0.1524" layer="1"/>
+<wire x1="28.575" y1="84.455" x2="33.02" y2="88.9" width="0.1524" layer="1"/>
+<wire x1="33.02" y1="88.9" x2="33.02" y2="92.71" width="0.1524" layer="1"/>
 </signal>
 <signal name="SCL">
@@
 <contactref element="U$2" pad="19/A5/SCL"/>
 <wire x1="40.64" y1="59.69" x2="54.61" y2="45.72" width="0.1524" layer="1"/>
-<wire x1="38.735" y1="59.69" x2="40.64" y2="59.69" width="0.1524" layer="1"/>
-<wire x1="27.94" y1="70.485" x2="38.735" y2="59.69" width="0.1524" layer="1"/>
-<wire x1="27.94" y1="71.12" x2="27.94" y2="70.485" width="0.1524" layer="1"/>
+<wire x1="40.64" y1="59.69" x2="38.735" y2="59.69" width="0.1524" layer="1"/>
+<wire x1="38.735" y1="59.69" x2="36.83" y2="61.595" width="0.1524" layer="1"/>
+<wire x1="36.83" y1="61.595" x2="36.83" y2="92.71" width="0.1524" layer="1"/>
+<wire x1="35.0774" y1="94.4626" x2="32.2326" y2="94.4626" width="0.1524" layer="1"/>
+<wire x1="32.2326" y1="94.4626" x2="30.48" y2="92.71" width="0.1524" layer="1"/>
+<wire x1="36.83" y1="92.71" x2="35.0774" y2="94.4626" width="0.1524" layer="1"/>
 </signal>
 <signal name="LED2">

Commit message: Updated comms testing board
Parts:
- added S3, S4: SWITCH_SLIDE_OS102011MS2QN1, GTOR - Active Components:OS102011MA1QN1
- added S5: PTS636_SL50_LFS, GTOR - Active Components:PTS636SL50LFS
- added X1: (no value), GTOR - Microfit Connector:43045-0400
- added X2: (no value), GTOR - Microfit Connector:43650-0300
- added X3: (no value), GTOR - Microfit Connector:43045-0600
- moved U$2 11.4 mm to (55.9, 41.9)
- moved LED2 11.4 mm to (25.4, 43.2)
- moved J1 9.92 mm to (1.27, 8.89)
- moved LED1 8.98 mm to (24.1, 11.4)
- moved R1 8.52 mm to (-2.54, 31.8)
- moved S1 8.03 mm to (30.5, 27.9)
- moved S2 7.62 mm to (20.3, 27.9)
- moved U$1 7.62 mm to (55.9, 11.4)
- moved R2 7.62 mm to (-2.54, 76.2)
- moved J2 6.48 mm to (1.27, 54.6)
Connections:
- new net A1: U$2.17/A3, X2.P$2
- new net CS: U$2.10/CS, X3.P$5
- new net DP: S5.1, U$2.2
- new net DP2: S5.2, U$2.3/CANTX
- new net MISO: U$2.12/MISO, X3.P$3
- new net MOSI: U$2.11/MOSI, X3.P$2
- new net R4: S4.2, U$2.7
- new net SCK: U$2.13/SCK, X3.P$4
- new net T4: S4.1, U$3.2
- net 3V3: now also X1.P$1, X2.P$1, X3.P$1
- net GND: now also X1.P$4, X2.P$3, X3.P$6
- net R3: now also S3.2; no longer U$2.8
- net SCL: now also X1.P$3
- net SDA: now also X1.P$2
- net T3: now also S3.1, U$2.8; no longer U$2.7, U$3.2
Routing:
- net 3V3: track 181.9 -> 0.00 mm
- net SDA: track 58.6 -> 149.4 mm, vias 0 -> 2
- net A1: track 0.00 -> 88.7 mm, vias 0 -> 1
- net SCL: track 63.3 -> 146.8 mm, vias 0 -> 1
- net MOSI: track 0.00 -> 79.8 mm
- net MISO: track 0.00 -> 73.0 mm
- net SCK: track 0.00 -> 61.4 mm, vias 0 -> 1
- net CS: track 0.00 -> 53.9 mm, vias 0 -> 2
- net T4: track 0.00 -> 45.5 mm
- net R4: track 0.00 -> 28.7 mm
- net DP2: track 0.00 -> 19.2 mm
- net P2: track 60.9 -> 79.5 mm, vias 0 -> 2
- net R3: track 24.4 -> 40.8 mm
- net P1: track 51.9 -> 62.6 mm, vias 0 -> 1
- net C2: track 34.7 -> 45.0 mm, vias 0 -> 1
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- added copper zone on layer 1, net 3V3
Other:
- board size 76.2 x 100 mm -> 82.5 x 116.5 mm
- board text added: "CS: Main 10"
- board text added: "I2C: MAIN 18,19"
- board text added: "I2C: MAIN 19, 18"
- board text added: "M14"
- board text added: "M16"
- board text added: "M2S"
- board text added: "M2X"
- board text added: "MAIN DP2"
- board text added: "MAIN DP3"
- board text added: "MAIN TEENSY TO XBEE TOGGLE"
- board text added: "MRX"
- board text added: "MTX"
- board text added: "Main17\"
- board text added: "S14"
- board text added: "S16"
- board text added: "S2M"
- board text added: "SRX"
- board text added: "STX"
- board text added: "X2M"
- board text added: "XBEE RX"
- board text added: "XBEE TX"
- board text removed: "R1 & T2"
- board text removed: "T1 & R2"
