File: Misc_Projects/Shock_Dyno/ShockDyno2022/Shock Dyno PCB/shock dyno.brd (EAGLE design)
At the start: 100 x 83.8 mm, 31 parts, among them IC1 ADS8332IBPWR, J1 1985195, K1 T9GS1L14-5, U1 REF5040AIDR

Commit message: final touches to shock dyno PCB part 2
Parts:
- added C5, C6: (no value), GTOR - Passive Components:C0603
- moved C4 0.32 mm to (42.5, 61.6)
Connections:
- removed net COIL1: D1.1, K1.2
- net +3V3: now also C6.1
- net GND: now also C5.2, C6.2
- net VCC: now also C5.1, D1.1, K1.2
Routing:
- net VCC: track 266.4 -> 298.3 mm
- net COIL1: track 11.4 -> 0.00 mm
- net GND: track 82.9 -> 90.7 mm, vias 3 -> 8
- net LDS_IN: track 135.2 -> 130.0 mm
- net +3V3: track 236.5 -> 233.4 mm
- net DIGITALPIN#1: track 3.81 -> 6.77 mm
- net COIL2: track 22.1 -> 21.1 mm
- net N$28: track 0.00 -> 0.65 mm
- net N$10: track 2.78 -> 3.42 mm

Commit message: final touches to shock dyno PCB part 3
Parts:
- C5, C6: value (none) -> 0.1μF
Changed lines of the file:
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@@
 <attribute name="VALUE" x="43.815" y="67.945" size="1.27" layer="27" rot="R180"/>
 </element>
-<element name="C5" library="GTOR - Passive Components" package="C0603" package3d_urn="urn:adsk.eagle:package:23616/2" value="" x="39.37" y="69.85" smashed="yes">
+<element name="C5" library="GTOR - Passive Components" package="C0603" package3d_urn="urn:adsk.eagle:package:23616/2" value="0.1μF" x="39.37" y="69.85" smashed="yes">
 <attribute name="NAME" x="38.1" y="70.8025" size="1.27" layer="25"/>
 <attribute name="POPULARITY" value="73" x="39.37" y="69.85" size="1.778" layer="27" display="off"/>
@@
 <attribute name="VALUE" x="38.735" y="67.945" size="1.27" layer="27"/>
 </element>
-<element name="C6" library="GTOR - Passive Components" package="C0603" package3d_urn="urn:adsk.eagle:package:23616/2" value="" x="48.26" y="60.96" smashed="yes" rot="R90">
+<element name="C6" library="GTOR - Passive Components" package="C0603" package3d_urn="urn:adsk.eagle:package:23616/2" value="0.1μF" x="48.26" y="60.96" smashed="yes" rot="R90">
 <attribute name="NAME" x="50.4825" y="59.69" size="1.27" layer="25" rot="R90"/>
 <attribute name="POPULARITY" value="73" x="48.26" y="60.96" size="1.778" layer="27" rot="R90" display="off"/>

Commit message: oriented load cell connector correctly
Connections:
- net GND: now also LOAD_CELL.3; no longer LOAD_CELL.2
- net LOAD_CELL: now also LOAD_CELL.2; no longer LOAD_CELL.3
- net VCC: now also LOAD_CELL.1; no longer LOAD_CELL.4
Routing:
- net GND: track 90.7 -> 106.0 mm, vias 8 -> 9
- net VCC: track 298.3 -> 294.4 mm
- net LOAD_CELL: track 43.6 -> 46.1 mm
Changed lines of the file:
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@@
 <contactref element="IC1" pad="19"/>
 <contactref element="C4" pad="1"/>
-<contactref element="LOAD_CELL" pad="2"/>
 <contactref element="LDS_IN" pad="3"/>
 <contactref element="JP1" pad="14"/>
@@
 <wire x1="24.765" y1="77.4" x2="24.8675" y2="77.5025" width="0.1524" layer="1"/>
 <wire x1="24.8675" y1="77.5025" x2="24.8675" y2="80.645" width="0.1524" layer="1"/>
-<wire x1="5.08" y1="71.12" x2="11.36" y2="77.4" width="0.1524" layer="1"/>
-<wire x1="11.36" y1="77.4" x2="24.765" y2="77.4" width="0.1524" layer="1"/>
+<wire x1="24.765" y1="77.4" x2="12.7" y2="77.4" width="0.1524" layer="1"/>
+<wire x1="12.7" y1="77.4" x2="11.36" y2="77.4" width="0.1524" layer="1"/>
 <wire x1="41.91" y1="14.82" x2="43.6" y2="16.51" width="0.1524" layer="1"/>
 <wire x1="43.6" y1="16.51" x2="46.99" y2="16.51" width="0.1524" layer="1"/>
@@
 <via x="41.91" y="69.85" extent="1-16" drill="0.35"/>
 <wire x1="40.22" y1="69.85" x2="41.91" y2="69.85" width="0.1524" layer="1"/>
+<contactref element="LOAD_CELL" pad="3"/>
+<wire x1="11.36" y1="77.4" x2="6.8326" y2="72.8726" width="0.1524" layer="1"/>
+<wire x1="5.08" y1="68.957075" x2="5.08" y2="68.58" width="0.1524" layer="1"/>
+<wire x1="6.8326" y1="72.8726" x2="6.8326" y2="70.709675" width="0.1524" layer="1"/>
+<wire x1="6.8326" y1="70.709675" x2="5.08" y2="68.957075" width="0.1524" layer="1"/>
+<wire x1="6.8326" y1="65.629675" x2="6.8326" y2="66.450325" width="0.1524" layer="1"/>
+<wire x1="5.08" y1="58.42" x2="5.08" y2="63.877075" width="0.1524" layer="1"/>
+<wire x1="5.08" y1="68.202925" x2="5.08" y2="68.58" width="0.1524" layer="1"/>
+<wire x1="5.08" y1="63.877075" x2="6.8326" y2="65.629675" width="0.1524" layer="1"/>
+<wire x1="6.8326" y1="66.450325" x2="5.08" y2="68.202925" width="0.1524" layer="1"/>
+<via x="12.7" y="76.2" extent="1-16" drill="0.35"/>
+<wire x1="12.7" y1="76.2" x2="12.7" y2="77.4" width="0.1524" layer="1"/>
 </signal>
 <signal name="+3V3">
@@
 <signal name="LOAD_CELL">
 <contactref element="U$1" pad="12"/>
-<contactref element="LOAD_CELL" pad="3"/>
 <wire x1="15.621" y1="33.8778125" x2="15.4870875" y2="33.7439" width="0.1524" layer="1"/>
 <wire x1="15.875" y1="34.4678" x2="15.621" y2="34.2138" width="0.1524" layer="1"/>
@@
 <wire x1="5.693525" y1="54.8894" x2="3.907675" y2="54.8894" width="0.1524" layer="1"/>
 <wire x1="6.8326" y1="53.750325" x2="5.693525" y2="54.8894" width="0.1524" layer="1"/>
-<wire x1="3.3274" y1="66.8274" x2="5.08" y2="68.58" width="0.1524" layer="1"/>
 <wire x1="6.35" y1="41.7518125" x2="6.35" y2="52.447075" width="0.1524" layer="1"/>
-<wire x1="3.3274" y1="55.469675" x2="3.3274" y2="66.8274" width="0.1524" layer="1"/>
+<contactref element="LOAD_CELL" pad="2"/>
+<wire x1="3.3274" y1="69.3674" x2="5.08" y2="71.12" width="0.1524" layer="1"/>
+<wire x1="3.3274" y1="55.469675" x2="3.3274" y2="69.3674" width="0.1524" layer="1"/>
 </signal>
 <signal name="N$9">
@@
 <contactref element="C3" pad="2"/>
 <contactref element="IC1" pad="17"/>
-<contactref element="LOAD_CELL" pad="4"/>
 <contactref element="LDS_IN" pad="1"/>
 <contactref element="U$2" pad="VIN"/>
@@
 <wire x1="26.5675" y1="78.1375" x2="26.5675" y2="80.01" width="0.1524" layer="1"/>
 <wire x1="26.5675" y1="80.01" x2="26.5675" y2="80.645" width="0.1524" layer="1"/>
-<wire x1="6.8326" y1="68.169675" x2="6.8326" y2="68.990325" width="0.1524" layer="1"/>
-<wire x1="3.907675" y1="70.1294" x2="3.3274" y2="70.709675" width="0.1524" layer="1"/>
-<wire x1="5.08" y1="66.04" x2="5.08" y2="66.417075" width="0.1524" layer="1"/>
-<wire x1="3.3274" y1="74.070325" x2="3.81" y2="74.552925" width="0.1524" layer="1"/>
-<wire x1="3.81" y1="74.552925" x2="3.81" y2="74.93" width="0.1524" layer="1"/>
-<wire x1="5.08" y1="66.417075" x2="6.8326" y2="68.169675" width="0.1524" layer="1"/>
-<wire x1="6.8326" y1="68.990325" x2="5.693525" y2="70.1294" width="0.1524" layer="1"/>
-<wire x1="5.693525" y1="70.1294" x2="3.907675" y2="70.1294" width="0.1524" layer="1"/>
-<wire x1="3.3274" y1="70.709675" x2="3.3274" y2="74.070325" width="0.1524" layer="1"/>
 <wire x1="25.5121875" y1="81.3736" x2="25.6461" y2="81.2396875" width="0.1524" layer="1"/>
 <wire x1="25.6461" y1="81.2396875" x2="25.6461" y2="80.9314" width="0.1524" layer="1"/>
 <wire x1="25.6461" y1="80.9314" x2="26.5675" y2="80.01" width="0.1524" layer="1"/>
-<wire x1="3.81" y1="74.93" x2="10.2536" y2="81.3736" width="0.1524" layer="1"/>
-<wire x1="10.2536" y1="81.3736" x2="25.5121875" y2="81.3736" width="0.1524" layer="1"/>
+<wire x1="25.5121875" y1="81.3736" x2="10.2536" y2="81.3736" width="0.1524" layer="1"/>
 <wire x1="93.98" y1="57.15" x2="93.98" y2="60.96" width="0.3048" layer="1"/>
 <wire x1="93.98" y1="57.15" x2="90.8685" y2="54.0385" width="0.3048" layer="1"/>
@@
 <wire x1="5.08" y1="53.34" x2="4.1275" y2="53.34" width="0.3048" layer="16"/>
 <wire x1="4.1275" y1="53.34" x2="2.54" y2="54.9275" width="0.3048" layer="16"/>
-<wire x1="2.54" y1="54.9275" x2="2.54" y2="63.5" width="0.3048" layer="16"/>
-<wire x1="2.54" y1="63.5" x2="5.08" y2="66.04" width="0.3048" layer="16"/>
 <contactref element="D1" pad="1"/>
 <contactref element="K1" pad="2"/>
@@
 <wire x1="46.99" y1="33.02" x2="58.36" y2="33.02" width="0.3048" layer="1"/>
 <wire x1="58.36" y1="33.02" x2="60.2615" y2="33.02" width="0.3048" layer="1"/>
+<contactref element="LOAD_CELL" pad="1"/>
+<wire x1="10.2536" y1="81.3736" x2="5.08" y2="76.2" width="0.1524" layer="1"/>
+<wire x1="5.08" y1="76.2" x2="5.08" y2="73.66" width="0.1524" layer="1"/>
+<wire x1="2.54" y1="71.12" x2="5.08" y2="73.66" width="0.3048" layer="16"/>
+<wire x1="2.54" y1="54.9275" x2="2.54" y2="71.12" width="0.3048" layer="16"/>
 </signal>
 <signal name="MISO">
