File: Misc_Projects/Strain_Gauges/Strain Gauge Amplifier.sch (EAGLE design)
At the start: 17 parts, among them IC1 INS_OPAMP_AD8221, J1 1985218, J3 1985218

Commit message: Added optional headers for strain gauge breakout
Parts:
- added JP2, JP3: (no value), GTOR - Connectors:PINHD-1X4
Connections:
- net 5V: now also JP2.1, JP3.1
- net A+: now also JP2.2
- net A-: now also JP2.4
- net GND: now also JP2.3, JP3.3
- net VOUT: now also JP3.2
Changed lines of the file:
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@@
 <part name="R6" library="GTOR - Passive Components" deviceset="RES_SMD" device="R0603" package3d_urn="urn:adsk.eagle:package:23555/3" value="86.6k"/>
 <part name="JP1" library="GTOR - Connectors" deviceset="PINHD-1X4" device="" package3d_urn="urn:adsk.eagle:package:22407/2"/>
+<part name="JP2" library="GTOR - Connectors" deviceset="PINHD-1X4" device="" package3d_urn="urn:adsk.eagle:package:22407/2"/>
+<part name="JP3" library="GTOR - Connectors" deviceset="PINHD-1X4" device="" package3d_urn="urn:adsk.eagle:package:22407/2"/>
 </parts>
 <sheets>
@@
 <attribute name="VALUE" x="146.05" y="-5.08" size="1.778" layer="96"/>
 </instance>
+<instance part="JP2" gate="A" x="30.48" y="10.16" smashed="yes">
+<attribute name="NAME" x="24.13" y="18.415" size="1.778" layer="95"/>
+<attribute name="VALUE" x="24.13" y="2.54" size="1.778" layer="96"/>
+</instance>
+<instance part="JP3" gate="A" x="238.76" y="0" smashed="yes">
+<attribute name="NAME" x="232.41" y="8.255" size="1.778" layer="95"/>
+<attribute name="VALUE" x="232.41" y="-7.62" size="1.778" layer="96"/>
+</instance>
 </instances>
 <busses>
@@
 <wire x1="149.86" y1="5.08" x2="139.7" y2="5.08" width="0.1524" layer="91"/>
 <label x="139.7" y="5.08" size="1.778" layer="95"/>
+</segment>
+<segment>
+<pinref part="JP2" gate="A" pin="2"/>
+<wire x1="27.94" y1="12.7" x2="17.78" y2="12.7" width="0.1524" layer="91"/>
+<label x="17.78" y="12.7" size="1.778" layer="95"/>
 </segment>
 </net>
@@
 <label x="139.7" y="0" size="1.778" layer="95"/>
 </segment>
+<segment>
+<pinref part="JP2" gate="A" pin="4"/>
+<wire x1="27.94" y1="7.62" x2="17.78" y2="7.62" width="0.1524" layer="91"/>
+<label x="17.78" y="7.62" size="1.778" layer="95"/>
+</segment>
 </net>
 <net name="5V" class="0">
@@
 <wire x1="149.86" y1="7.62" x2="139.7" y2="7.62" width="0.1524" layer="91"/>
 <label x="139.7" y="7.62" size="1.778" layer="95"/>
+</segment>
+<segment>
+<pinref part="JP2" gate="A" pin="1"/>
+<wire x1="27.94" y1="15.24" x2="17.78" y2="15.24" width="0.1524" layer="91"/>
+<label x="17.78" y="15.24" size="1.778" layer="95"/>
+</segment>
+<segment>
+<pinref part="JP3" gate="A" pin="1"/>
+<wire x1="236.22" y1="5.08" x2="226.06" y2="5.08" width="0.1524" layer="91"/>
+<label x="226.06" y="5.08" size="1.778" layer="95"/>
 </segment>
 </net>
@@
 <label x="139.7" y="2.54" size="1.778" layer="95"/>
 </segment>
+<segment>
+<pinref part="JP2" gate="A" pin="3"/>
+<wire x1="27.94" y1="10.16" x2="17.78" y2="10.16" width="0.1524" layer="91"/>
+<label x="17.78" y="10.16" size="1.778" layer="95"/>
+</segment>
+<segment>
+<pinref part="JP3" gate="A" pin="3"/>
+<wire x1="236.22" y1="0" x2="226.06" y2="0" width="0.1524" layer="91"/>
+<label x="226.06" y="0" size="1.778" layer="95"/>
+</segment>
 </net>
 <net name="N$2" class="0">
@@
 <label x="187.96" y="20.32" size="1.778" layer="95"/>
 </segment>
-</net>
+<segment>
+<pinref part="JP3" gate="A" pin="2"/>
+<wire x1="236.22" y1="2.54" x2="226.06" y2="2.54" width="0.1524" layer="91"/>
+<label x="226.06" y="2.54" size="1.778" layer="95"/>
+</segment>
+</net>

Commit message: changed connectors on strain gauge amplifier to microfit
Parts:
- removed J1, J3: 1985218, GTOR - Connectors:1985218
- added X1, X2: (no value), GTOR - Microfit Connector:HEADER_POS4_43045-0401
Connections:
- removed net N$15: J3.4
- net 5V: now also X1.1, X2.1; no longer J1.1, J3.1
- net A+: now also X1.2; no longer J1.2
- net A-: now also X1.3; no longer J1.4
- net GND: now also X1.4, X2.4; no longer J1.3, J3.3
- net VOUT: now also X2.2; no longer J3.2
Other:
- moved on the sheet: JP1
Changed lines of the file:
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@@
 </classes>
 <parts>
-<part name="J1" library="GTOR - Connectors" deviceset="1985218" device=""/>
 <part name="R1" library="GTOR - Passive Components" deviceset="RES_SMD" device="R1206" package3d_urn="urn:adsk.eagle:package:23540/2"/>
 <part name="R2" library="GTOR - Passive Components" deviceset="RES_SMD" device="R1206" package3d_urn="urn:adsk.eagle:package:23540/2"/>
@@
 <part name="R4" library="GTOR - Passive Components" deviceset="RES_SMD" device="R1206" package3d_urn="urn:adsk.eagle:package:23540/2"/>
 <part name="IC1" library="GTOR - Active Components" deviceset="INS_OPAMP_AD8221" device=""/>
-<part name="J3" library="GTOR - Connectors" deviceset="1985218" device=""/>
 <part name="C1" library="GTOR - Passive Components" deviceset="CAP_THT" device="E2-5" package3d_urn="urn:adsk.eagle:package:23346/2" value="10u"/>
 <part name="PS1" library="GTOR - Active Components" deviceset="REF_2V5_MCP1501T-25E_SN" device=""/>
@@
 <part name="JP2" library="GTOR - Connectors" deviceset="PINHD-1X4" device="" package3d_urn="urn:adsk.eagle:package:22407/2"/>
 <part name="JP3" library="GTOR - Connectors" deviceset="PINHD-1X4" device="" package3d_urn="urn:adsk.eagle:package:22407/2"/>
+<part name="X1" library="GTOR - Microfit Connector" deviceset="HEADER_POS4_?" device="43045-0401"/>
+<part name="X2" library="GTOR - Microfit Connector" deviceset="HEADER_POS4_?" device="43045-0401"/>
 </parts>
 <sheets>
@@
 </plain>
 <instances>
-<instance part="J1" gate="G$1" x="2.54" y="33.02" smashed="yes">
-<attribute name="NAME" x="19.05" y="40.64" size="1.778" layer="95" align="center-left"/>
-<attribute name="VALUE" x="19.05" y="38.1" size="1.778" layer="96" align="center-left"/>
-</instance>
 <instance part="R1" gate="G$1" x="48.26" y="33.02" smashed="yes" rot="R90">
 <attribute name="NAME" x="46.7614" y="29.21" size="1.778" layer="95" rot="R90"/>
@@
 <attribute name="VALUE" x="181.61" y="27.94" size="1.778" layer="96" align="center-left"/>
 </instance>
-<instance part="J3" gate="G$1" x="193.04" y="0" smashed="yes">
-<attribute name="NAME" x="209.55" y="7.62" size="1.778" layer="95" align="center-left"/>
-<attribute name="VALUE" x="209.55" y="5.08" size="1.778" layer="96" align="center-left"/>
-</instance>
 <instance part="C1" gate="G$1" x="205.74" y="20.32" smashed="yes">
 <attribute name="NAME" x="206.756" y="20.955" size="1.778" layer="95"/>
@@
 <attribute name="VALUE" x="76.962" y="3.81" size="1.778" layer="96" rot="R90"/>
 </instance>
-<instance part="JP1" gate="A" x="152.4" y="2.54" smashed="yes">
-<attribute name="NAME" x="146.05" y="10.795" size="1.778" layer="95"/>
-<attribute name="VALUE" x="146.05" y="-5.08" size="1.778" layer="96"/>
+<instance part="JP1" gate="A" x="152.4" y="0" smashed="yes">
+<attribute name="NAME" x="146.05" y="8.255" size="1.778" layer="95"/>
+<attribute name="VALUE" x="146.05" y="-7.62" size="1.778" layer="96"/>
 </instance>
 <instance part="JP2" gate="A" x="30.48" y="10.16" smashed="yes">
@@
 <attribute name="NAME" x="232.41" y="8.255" size="1.778" layer="95"/>
 <attribute name="VALUE" x="232.41" y="-7.62" size="1.778" layer="96"/>
+</instance>
+<instance part="X1" gate="G$1" x="27.94" y="30.48" smashed="yes">
+<attribute name="VALUE" x="26.67" y="22.86" size="1.778" layer="96"/>
+<attribute name="NAME" x="26.67" y="38.862" size="1.778" layer="95"/>
+</instance>
+<instance part="X2" gate="G$1" x="236.22" y="20.32" smashed="yes">
+<attribute name="VALUE" x="234.95" y="12.7" size="1.778" layer="96"/>
+<attribute name="NAME" x="234.95" y="28.702" size="1.778" layer="95"/>
 </instance>
 </instances>
@@
 </segment>
 <segment>
-<pinref part="J1" gate="G$1" pin="2"/>
-<wire x1="2.54" y1="33.02" x2="-5.08" y2="33.02" width="0.1524" layer="91"/>
-<label x="-5.08" y="33.02" size="1.778" layer="95"/>
-</segment>
-<segment>
 <pinref part="IC1" gate="G$1" pin="+IN"/>
 <wire x1="157.48" y1="15.24" x2="149.86" y2="15.24" width="0.1524" layer="91"/>
@@
 <segment>
 <pinref part="JP1" gate="A" pin="2"/>
-<wire x1="149.86" y1="5.08" x2="139.7" y2="5.08" width="0.1524" layer="91"/>
-<label x="139.7" y="5.08" size="1.778" layer="95"/>
+<wire x1="149.86" y1="2.54" x2="139.7" y2="2.54" width="0.1524" layer="91"/>
+<label x="139.7" y="2.54" size="1.778" layer="95"/>
 </segment>
 <segment>
@@
 <wire x1="27.94" y1="12.7" x2="17.78" y2="12.7" width="0.1524" layer="91"/>
 <label x="17.78" y="12.7" size="1.778" layer="95"/>
+</segment>
+<segment>
+<pinref part="X1" gate="G$1" pin="2"/>
+<wire x1="22.86" y1="33.02" x2="15.24" y2="33.02" width="0.1524" layer="91"/>
+<label x="15.24" y="33.02" size="1.778" layer="95"/>
 </segment>
 </net>
@@
 </segment>
 <segment>
-<pinref part="J1" gate="G$1" pin="4"/>
-<wire x1="2.54" y1="30.48" x2="-5.08" y2="30.48" width="0.1524" layer="91"/>
-<label x="-5.08" y="30.48" size="1.778" layer="95"/>
-</segment>
-<segment>
 <pinref part="IC1" gate="G$1" pin="-IN"/>
 <wire x1="157.48" y1="22.86" x2="149.86" y2="22.86" width="0.1524" layer="91"/>
@@
 <segment>
 <pinref part="JP1" gate="A" pin="4"/>
-<wire x1="149.86" y1="0" x2="139.7" y2="0" width="0.1524" layer="91"/>
-<label x="139.7" y="0" size="1.778" layer="95"/>
+<wire x1="149.86" y1="-2.54" x2="139.7" y2="-2.54" width="0.1524" layer="91"/>
+<label x="139.7" y="-2.54" size="1.778" layer="95"/>
 </segment>
 <segment>
@@
 <wire x1="27.94" y1="7.62" x2="17.78" y2="7.62" width="0.1524" layer="91"/>
 <label x="17.78" y="7.62" size="1.778" layer="95"/>
+</segment>
+<segment>
+<pinref part="X1" gate="G$1" pin="3"/>
+<wire x1="22.86" y1="30.48" x2="15.24" y2="30.48" width="0.1524" layer="91"/>
+<label x="15.24" y="30.48" size="1.778" layer="95"/>
 </segment>
 </net>
@@
 </segment>
 <segment>
-<pinref part="J1" gate="G$1" pin="1"/>
-<wire x1="22.86" y1="33.02" x2="30.48" y2="33.02" width="0.1524" layer="91"/>
-<label x="25.4" y="33.02" size="1.778" layer="95"/>
-</segment>
-<segment>
 <pinref part="IC1" gate="G$1" pin="+VS"/>
 <label x="187.96" y="22.86" size="1.778" layer="95"/>
@@
 <wire x1="213.36" y1="22.86" x2="205.74" y2="22.86" width="0.1524" layer="91"/>
 <junction x="205.74" y="22.86"/>
-</segment>
-<segment>
-<pinref part="J3" gate="G$1" pin="1"/>
-<wire x1="213.36" y1="0" x2="220.98" y2="0" width="0.1524" layer="91"/>
-<label x="215.9" y="0" size="1.778" layer="95"/>
 </segment>
 <segment>
@@
 <segment>
 <pinref part="JP1" gate="A" pin="1"/>
-<wire x1="149.86" y1="7.62" x2="139.7" y2="7.62" width="0.1524" layer="91"/>
-<label x="139.7" y="7.62" size="1.778" layer="95"/>
+<wire x1="149.86" y1="5.08" x2="139.7" y2="5.08" width="0.1524" layer="91"/>
+<label x="139.7" y="5.08" size="1.778" layer="95"/>
 </segment>
 <segment>
@@
 <wire x1="236.22" y1="5.08" x2="226.06" y2="5.08" width="0.1524" layer="91"/>
 <label x="226.06" y="5.08" size="1.778" layer="95"/>
+</segment>
+<segment>
+<pinref part="X1" gate="G$1" pin="1"/>
+<wire x1="22.86" y1="35.56" x2="15.24" y2="35.56" width="0.1524" layer="91"/>
+<label x="15.24" y="35.56" size="1.778" layer="95"/>
+</segment>
+<segment>
+<pinref part="X2" gate="G$1" pin="1"/>
+<wire x1="231.14" y1="25.4" x2="223.52" y2="25.4" width="0.1524" layer="91"/>
+<label x="223.52" y="25.4" size="1.778" layer="95"/>
 </segment>
 </net>
@@
 </segment>
 <segment>
-<pinref part="J1" gate="G$1" pin="3"/>
-<wire x1="22.86" y1="30.48" x2="30.48" y2="30.48" width="0.1524" layer="91"/>
-<label x="25.4" y="30.48" size="1.778" layer="95"/>
-</segment>
-<segment>
 <pinref part="IC1" gate="G$1" pin="-VS"/>
 <label x="187.96" y="15.24" size="1.778" layer="95"/>
@@
 <wire x1="205.74" y1="15.24" x2="213.36" y2="15.24" width="0.1524" layer="91"/>
 <junction x="205.74" y="15.24"/>
-</segment>
-<segment>
-<pinref part="J3" gate="G$1" pin="3"/>
-<wire x1="213.36" y1="-2.54" x2="220.98" y2="-2.54" width="0.1524" layer="91"/>
-<label x="215.9" y="-2.54" size="1.778" layer="95"/>
 </segment>
 <segment>
@@
 <segment>
 <pinref part="JP1" gate="A" pin="3"/>
-<wire x1="149.86" y1="2.54" x2="139.7" y2="2.54" width="0.1524" layer="91"/>
-<label x="139.7" y="2.54" size="1.778" layer="95"/>
+<wire x1="149.86" y1="0" x2="139.7" y2="0" width="0.1524" layer="91"/>
+<label x="139.7" y="0" size="1.778" layer="95"/>
 </segment>
 <segment>
@@
 <wire x1="236.22" y1="0" x2="226.06" y2="0" width="0.1524" layer="91"/>
 <label x="226.06" y="0" size="1.778" layer="95"/>
+</segment>
+<segment>
+<pinref part="X1" gate="G$1" pin="4"/>
+<wire x1="22.86" y1="27.94" x2="15.24" y2="27.94" width="0.1524" layer="91"/>
+<label x="15.24" y="27.94" size="1.778" layer="95"/>
+</segment>
+<segment>
+<pinref part="X2" gate="G$1" pin="4"/>
+<wire x1="231.14" y1="17.78" x2="223.52" y2="17.78" width="0.1524" layer="91"/>
+<label x="223.52" y="17.78" size="1.778" layer="95"/>
 </segment>
 </net>
@@
 <net name="VOUT" class="0">
 <segment>
-<pinref part="J3" gate="G$1" pin="2"/>
-<wire x1="193.04" y1="0" x2="185.42" y2="0" width="0.1524" layer="91"/>
-<label x="185.42" y="0" size="1.778" layer="95"/>
-</segment>
-<segment>
 <pinref part="IC1" gate="G$1" pin="VOUT"/>
 <wire x1="185.42" y1="20.32" x2="193.04" y2="20.32" width="0.1524" layer="91"/>
@@
 <label x="226.06" y="2.54" size="1.778" layer="95"/>
 </segment>
-</net>
-<net name="N$15" class="0">
-<segment>
-<pinref part="J3" gate="G$1" pin="4"/>
-<wire x1="193.04" y1="-2.54" x2="185.42" y2="-2.54" width="0.1524" layer="91"/>
-</segment>
-</net>
+<segment>
+<pinref part="X2" gate="G$1" pin="2"/>
+<wire x1="231.14" y1="22.86" x2="223.52" y2="22.86" width="0.1524" layer="91"/>
+<label x="223.52" y="22.86" size="1.778" layer="95"/>
+</segment>
+</net>
