File: Misc_Projects/Light_Gates/LightGateBoard2022/EndLightGate2022.brd (EAGLE design)
At the start: 57.1 x 49.5 mm, 8 parts, among them J1 TB005-762-02BE

Commit message: Light Gate Updates
Parts:
- removed IC1: (no value), GTOR - Active Components:TO-220
- removed X1: (no value), GTOR - Microfit Connector:43045-0600
- added IC2: (no value), GTOR - Active Components:TO-220-H
- added JP1: (no value), GTOR - Connectors:1X06
- moved X2 14.0 mm to (5.08, 26.7)
- moved R2 8.98 mm to (43.2, 41.9)
- moved R1 7.73 mm to (39.4, 41.9)
- moved U$2 5.08 mm to (24.1, 45.7)
- moved J1 3.51 mm to (42.4, 13.6)
Connections:
- net +3V3: now also JP1.6; no longer X1.P$6
- net +5V: now also IC2.3; no longer IC1.3
- net GND: now also IC2.2, JP1.5; no longer IC1.2, X1.P$5
- net INT: now also JP1.1; no longer X1.P$1
- net SCL: now also JP1.3; no longer X1.P$3
- net SDA: now also JP1.4; no longer X1.P$4
- net SHUT: now also JP1.2; no longer X1.P$2
- net VCC: now also IC2.1; no longer IC1.1
Routing:
- net OUTPUT: track 46.5 -> 26.6 mm
- net SHUT: track 28.7 -> 41.0 mm
- net SDA: track 61.6 -> 73.3 mm
- net +3V3: track 74.7 -> 86.3 mm
- net VCC: track 59.5 -> 51.4 mm
- net +5V: track 69.2 -> 75.2 mm
- net INT: track 25.2 -> 30.8 mm
- net SCL: track 82.2 -> 82.9 mm

Commit message: Fixed light gate end board
Other:
- board size 57.1 x 49.5 mm -> 57.1 x 50.8 mm
Changed lines of the file:
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@@
 <board>
 <plain>
-<wire x1="0" y1="0" x2="0" y2="49.53" width="0.1524" layer="20"/>
-<wire x1="0" y1="49.53" x2="57.15" y2="49.53" width="0.1524" layer="20"/>
-<wire x1="57.15" y1="49.53" x2="57.15" y2="0" width="0.1524" layer="20"/>
-<wire x1="57.15" y1="0" x2="0" y2="0" width="0.1524" layer="20"/>
+<wire x1="0" y1="0" x2="0" y2="50.8" width="0" layer="20"/>
+<wire x1="0" y1="50.8" x2="57.15" y2="50.8" width="0" layer="20"/>
+<wire x1="57.15" y1="50.8" x2="57.15" y2="0" width="0" layer="20"/>
+<wire x1="57.15" y1="0" x2="0" y2="0" width="0" layer="20"/>
 <text x="4.572" y="33.655" size="1.016" layer="21" rot="R90">End Light Gate V3
 Designed by:
 Param Pithadia</text>
-<hole x="2.54" y="46.736" drill="3.3"/>
-<hole x="42.418" y="29.083" drill="3.3"/>
-<hole x="54.864" y="2.159" drill="3.3"/>
+<hole x="3.175" y="44.45" drill="3.3"/>
+<hole x="53.975" y="6.35" drill="3.3"/>
+<hole x="3.175" y="6.35" drill="3.3"/>
+<hole x="53.975" y="44.45" drill="3.3"/>
 </plain>
 <attributes>
@@
 <wire x1="44.4722" y1="22.8822" x2="45.26" y2="23.67" width="0.1524" layer="1"/>
 <wire x1="44.4722" y1="20.0169625" x2="44.4722" y2="22.8822" width="0.1524" layer="1"/>
-<wire x1="42.418" y1="13.589" x2="42.418" y2="17.9627625" width="0.1524" layer="1"/>
-<wire x1="42.418" y1="17.9627625" x2="44.4722" y2="20.0169625" width="0.1524" layer="1"/>
+<wire x1="43.7090375" y1="19.2538" x2="43.97761875" y2="19.52238125" width="0.1524" layer="1"/>
+<wire x1="43.97761875" y1="19.52238125" x2="44.4722" y2="20.0169625" width="0.1524" layer="1"/>
+<wire x1="43.7090375" y1="19.2538" x2="42.418" y2="17.9627625" width="0.1524" layer="1"/>
+<wire x1="42.418" y1="17.9627625" x2="42.418" y2="13.589" width="0.1524" layer="1"/>
 </signal>
 <signal name="GND">
