File: Driver_Comms_Sender/Driver Message Board.sch (EAGLE design)
At the start: 14 parts, among them U1 XBEE_PRO_S3B

Commit message: Finalized PCB and started code
Other:
- note added: "VCC is 11.1 V"
- note removed: "VCC will be 7.4V"
Changed lines of the file:
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@@
 <sheet>
 <plain>
-<text x="81.28" y="40.64" size="1.778" layer="91">VCC will be 7.4V</text>
+<text x="86.36" y="35.56" size="1.778" layer="91">VCC is 11.1 V</text>
 </plain>
 <instances>
@@
 <pinref part="U$1" gate="G$1" pin="18/A4/SDA"/>
 <wire x1="58.42" y1="66.04" x2="73.66" y2="66.04" width="0.1524" layer="91"/>
-</segment>
-<segment>
+<label x="73.66" y="66.04" size="1.778" layer="95" xref="yes"/>
+</segment>
+<segment>
