File: Misc_Projects/Wireless_Comms/Comms_Testing/Eagle Files/CommsTestBoard/CommsTestBoard.sch (EAGLE design)
At the start: 18 parts, among them J1 1985205, J2 1985205

Commit message: Comms Test Board update
changed some stuff
Parts:
- U$2: value TEENSY_4.0_SIMPLE -> TEENSY_4.1_SIMPLE; device GTOR - Microcontroller:TEENSY_4.0_SIMPLE -> GTOR - Microcontroller:TEENSY_4.1_SIMPLE
- renumbered R1 to A2
Changed lines of the file:
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@@
 <parts>
 <part name="U$1" library="GTOR - Microcontroller" deviceset="TEENSY_4.0_SIMPLE" device=""/>
-<part name="U$2" library="GTOR - Microcontroller" deviceset="TEENSY_4.0_SIMPLE" device=""/>
-<part name="R1" library="GTOR - Passive Components" deviceset="POTENTIOMETER" device="" package3d_urn="urn:adsk.eagle:package:22726/1"/>
+<part name="U$2" library="GTOR - Microcontroller" deviceset="TEENSY_4.1_SIMPLE" device=""/>
+<part name="A2" library="GTOR - Passive Components" deviceset="POTENTIOMETER" device="" package3d_urn="urn:adsk.eagle:package:22726/1"/>
 <part name="R2" library="GTOR - Passive Components" deviceset="POTENTIOMETER" device="" package3d_urn="urn:adsk.eagle:package:22726/1"/>
 <part name="LED1" library="GTOR - Passive Components" deviceset="LED" device="-5MM"/>
@@
 <instances>
 <instance part="U$1" gate="G$1" x="7.62" y="50.8" smashed="yes"/>
-<instance part="U$2" gate="G$1" x="96.52" y="50.8" smashed="yes"/>
-<instance part="R1" gate="G$1" x="-12.7" y="12.7" smashed="yes">
+<instance part="U$2" gate="G$1" x="96.012" y="74.168" smashed="yes"/>
+<instance part="A2" gate="G$1" x="-12.7" y="12.7" smashed="yes">
 <attribute name="NAME" x="-18.669" y="8.89" size="1.778" layer="95" rot="R90"/>
 <attribute name="VALUE" x="-16.51" y="8.89" size="1.778" layer="96" rot="R90"/>
@@
 <segment>
 <pinref part="U$2" gate="G$1" pin="VIN"/>
-<wire x1="116.84" y1="63.5" x2="121.92" y2="63.5" width="0.1524" layer="91"/>
-<label x="119.38" y="63.5" size="1.778" layer="95"/>
+<wire x1="116.332" y1="86.868" x2="119.38" y2="86.868" width="0.1524" layer="91"/>
+<label x="116.84" y="86.868" size="1.778" layer="95"/>
 </segment>
 </net>
@@
 <segment>
 <pinref part="U$2" gate="G$1" pin="GND2"/>
-<wire x1="116.84" y1="60.96" x2="121.92" y2="60.96" width="0.1524" layer="91"/>
-<label x="119.38" y="60.96" size="1.778" layer="95"/>
+<wire x1="116.332" y1="84.328" x2="119.38" y2="84.328" width="0.1524" layer="91"/>
+<label x="116.84" y="84.328" size="1.778" layer="95"/>
 </segment>
 <segment>
@@
 </segment>
 <segment>
-<pinref part="R1" gate="G$1" pin="A"/>
+<pinref part="A2" gate="G$1" pin="A"/>
 <wire x1="-12.7" y1="7.62" x2="-12.7" y2="2.54" width="0.1524" layer="91"/>
 <label x="-17.78" y="2.54" size="1.778" layer="95"/>
@@
 </segment>
 <segment>
+<pinref part="X1" gate="G$1" pin="4"/>
+<wire x1="129.54" y1="-12.7" x2="124.46" y2="-12.7" width="0.1524" layer="91"/>
+<label x="121.92" y="-12.7" size="1.778" layer="95"/>
+</segment>
+<segment>
 <pinref part="X2" gate="G$1" pin="3"/>
 <wire x1="149.86" y1="-10.16" x2="144.78" y2="-10.16" width="0.1524" layer="91"/>
@@
 </segment>
 <segment>
-<pinref part="X1" gate="G$1" pin="4"/>
-<wire x1="129.54" y1="-12.7" x2="124.46" y2="-12.7" width="0.1524" layer="91"/>
-<label x="121.92" y="-12.7" size="1.778" layer="95"/>
-</segment>
-<segment>
 <pinref part="X3" gate="G$1" pin="6"/>
 <wire x1="170.18" y1="-15.24" x2="162.56" y2="-15.24" width="0.1524" layer="91"/>
@@
 <segment>
 <pinref part="U$2" gate="G$1" pin="3V3_LO"/>
-<wire x1="116.84" y1="58.42" x2="121.92" y2="58.42" width="0.1524" layer="91"/>
-<label x="119.38" y="58.42" size="1.778" layer="95"/>
-</segment>
-<segment>
-<pinref part="R1" gate="G$1" pin="E"/>
+<wire x1="116.332" y1="81.788" x2="119.38" y2="81.788" width="0.1524" layer="91"/>
+<label x="116.84" y="81.788" size="1.778" layer="95"/>
+</segment>
+<segment>
+<pinref part="A2" gate="G$1" pin="E"/>
 <wire x1="-12.7" y1="17.78" x2="-12.7" y2="20.32" width="0.1524" layer="91"/>
 <label x="-17.78" y="20.32" size="1.778" layer="95"/>
@@
 <segment>
 <pinref part="U$2" gate="G$1" pin="8/TX2"/>
-<wire x1="76.2" y1="40.64" x2="71.12" y2="40.64" width="0.1524" layer="91"/>
-<label x="71.12" y="40.64" size="1.778" layer="95"/>
+<wire x1="75.692" y1="64.008" x2="69.85" y2="64.008" width="0.1524" layer="91"/>
+<label x="69.85" y="64.008" size="1.778" layer="95"/>
 </segment>
 </net>
@@
 <segment>
 <pinref part="U$2" gate="G$1" pin="18/A4/SDA"/>
-<wire x1="116.84" y1="43.18" x2="121.92" y2="43.18" width="0.1524" layer="91"/>
-<label x="119.38" y="43.18" size="1.778" layer="95"/>
+<wire x1="116.332" y1="66.548" x2="119.38" y2="66.548" width="0.1524" layer="91"/>
+<label x="116.84" y="66.548" size="1.778" layer="95"/>
 </segment>
 <segment>
@@
 <segment>
 <pinref part="U$2" gate="G$1" pin="19/A5/SCL"/>
-<wire x1="116.84" y1="45.72" x2="121.92" y2="45.72" width="0.1524" layer="91"/>
-<label x="119.38" y="45.72" size="1.778" layer="95"/>
+<wire x1="116.332" y1="69.088" x2="119.38" y2="69.088" width="0.1524" layer="91"/>
+<label x="116.84" y="69.088" size="1.778" layer="95"/>
 </segment>
 <segment>
@@
 <segment>
 <pinref part="U$2" gate="G$1" pin="15/A1/RX3"/>
-<wire x1="116.84" y1="35.56" x2="121.92" y2="35.56" width="0.1524" layer="91"/>
-<label x="119.38" y="35.56" size="1.778" layer="95"/>
+<wire x1="116.332" y1="58.928" x2="119.38" y2="58.928" width="0.1524" layer="91"/>
+<label x="116.84" y="58.928" size="1.778" layer="95"/>
 </segment>
 <segment>
@@
 <net name="P1" class="0">
 <segment>
-<pinref part="R1" gate="G$1" pin="S"/>
+<pinref part="A2" gate="G$1" pin="S"/>
 <wire x1="-7.62" y1="12.7" x2="-5.08" y2="12.7" width="0.1524" layer="91"/>
 <label x="-7.62" y="12.7" size="1.778" layer="95"/>
@@
 <segment>
 <pinref part="U$2" gate="G$1" pin="16/A2/RX4"/>
-<wire x1="116.84" y1="38.1" x2="121.92" y2="38.1" width="0.1524" layer="91"/>
-<label x="119.38" y="38.1" size="1.778" layer="95"/>
+<wire x1="116.332" y1="61.468" x2="119.38" y2="61.468" width="0.1524" layer="91"/>
+<label x="116.84" y="61.468" size="1.778" layer="95"/>
 </segment>
 </net>
@@
 <segment>
 <pinref part="U$2" gate="G$1" pin="0/RX1"/>
-<wire x1="76.2" y1="60.96" x2="71.12" y2="60.96" width="0.1524" layer="91"/>
-<label x="71.12" y="60.96" size="1.778" layer="95"/>
+<wire x1="75.692" y1="84.328" x2="69.85" y2="84.328" width="0.1524" layer="91"/>
+<label x="69.85" y="84.328" size="1.778" layer="95"/>
 </segment>
 </net>
@@
 <segment>
 <pinref part="U$2" gate="G$1" pin="1/TX1"/>
-<wire x1="76.2" y1="58.42" x2="71.12" y2="58.42" width="0.1524" layer="91"/>
-<label x="71.12" y="58.42" size="1.778" layer="95"/>
+<wire x1="75.692" y1="81.788" x2="69.85" y2="81.788" width="0.1524" layer="91"/>
+<label x="69.85" y="81.788" size="1.778" layer="95"/>
 </segment>
 </net>
@@
 <segment>
 <pinref part="U$2" gate="G$1" pin="14/A0/TX3"/>
-<wire x1="116.84" y1="33.02" x2="121.92" y2="33.02" width="0.1524" layer="91"/>
-<label x="119.38" y="33.02" size="1.778" layer="95"/>
+<wire x1="116.332" y1="56.388" x2="119.38" y2="56.388" width="0.1524" layer="91"/>
+<label x="116.84" y="56.388" size="1.778" layer="95"/>
 </segment>
 <segment>
@@
 <segment>
 <pinref part="U$2" gate="G$1" pin="7/RX2"/>
-<wire x1="76.2" y1="43.18" x2="71.12" y2="43.18" width="0.1524" layer="91"/>
-<label x="71.12" y="43.18" size="1.778" layer="95"/>
+<wire x1="75.692" y1="66.548" x2="69.85" y2="66.548" width="0.1524" layer="91"/>
+<label x="69.85" y="66.548" size="1.778" layer="95"/>
 </segment>
 </net>
@@
 <segment>
 <pinref part="U$2" gate="G$1" pin="17/A3/TX4"/>
-<wire x1="116.84" y1="40.64" x2="124.46" y2="40.64" width="0.1524" layer="91"/>
-<label x="121.92" y="40.64" size="1.778" layer="95"/>
+<wire x1="116.332" y1="64.008" x2="119.888" y2="63.754" width="0.1524" layer="91"/>
+<label x="119.38" y="64.008" size="1.778" layer="95"/>
 </segment>
 </net>
@@
 <segment>
 <pinref part="U$2" gate="G$1" pin="11/MOSI"/>
-<wire x1="76.2" y1="33.02" x2="71.12" y2="33.02" width="0.1524" layer="91"/>
-<label x="71.12" y="33.02" size="1.778" layer="95"/>
+<wire x1="75.692" y1="56.388" x2="69.85" y2="56.388" width="0.1524" layer="91"/>
+<label x="69.85" y="56.388" size="1.778" layer="95"/>
 </segment>
 </net>
@@
 <segment>
 <pinref part="U$2" gate="G$1" pin="13/SCK"/>
-<wire x1="116.84" y1="30.48" x2="124.46" y2="30.48" width="0.1524" layer="91"/>
-<label x="121.92" y="30.48" size="1.778" layer="95"/>
+<wire x1="116.332" y1="53.848" x2="119.634" y2="53.848" width="0.1524" layer="91"/>
+<label x="119.38" y="53.848" size="1.778" layer="95"/>
 </segment>
 </net>
@@
 <segment>
 <pinref part="U$2" gate="G$1" pin="10/CS"/>
-<wire x1="76.2" y1="35.56" x2="71.12" y2="35.56" width="0.1524" layer="91"/>
-<label x="71.12" y="35.56" size="1.778" layer="95"/>
+<wire x1="75.692" y1="58.928" x2="69.85" y2="58.928" width="0.1524" layer="91"/>
+<label x="69.85" y="58.928" size="1.778" layer="95"/>
 </segment>
 </net>
@@
 <segment>
 <pinref part="U$2" gate="G$1" pin="12/MISO"/>
-<wire x1="76.2" y1="30.48" x2="71.12" y2="30.48" width="0.1524" layer="91"/>
-<label x="71.12" y="30.48" size="1.778" layer="95"/>
+<wire x1="75.692" y1="53.848" x2="69.85" y2="53.848" width="0.1524" layer="91"/>
+<label x="69.85" y="53.848" size="1.778" layer="95"/>
 </segment>
 <segment>
@@
 <segment>
 <pinref part="U$2" gate="G$1" pin="2"/>
-<wire x1="76.2" y1="55.88" x2="71.12" y2="55.88" width="0.1524" layer="91"/>
-<label x="71.12" y="55.88" size="1.778" layer="95"/>
+<wire x1="75.692" y1="79.248" x2="69.85" y2="79.248" width="0.1524" layer="91"/>
+<label x="69.85" y="79.248" size="1.778" layer="95"/>
 </segment>
 <segment>
@@
 <segment>
 <pinref part="U$2" gate="G$1" pin="3"/>
-<wire x1="76.2" y1="53.34" x2="71.12" y2="53.34" width="0.1524" layer="91"/>
-<label x="71.12" y="53.34" size="1.778" layer="95"/>
-</segment>
-<segment>
+<wire x1="75.692" y1="76.708" x2="69.85" y2="76.708" width="0.1524" layer="91"/>
+<label x="69.85" y="76.708" size="1.778" layer="95"/>
+</segment>
+<segment>
