File: Misc_Projects/Wireless_Comms/Comms_Testing/Eagle Files/CommsTestBoard/CommsTestBoard.brd (EAGLE design)
At the start: 82.5 x 116.5 mm, 18 parts, among them J1 1985205, J2 1985205

Commit message: Comms Test Board update
changed some stuff
Parts:
- U$2: value TEENSY_4.0_SIMPLE -> TEENSY_4.1_SIMPLE; device GTOR - Microcontroller:TEENSY_4.0_SIMPLE -> GTOR - Microcontroller:TEENSY_4.1_SIMPLE
- moved LED2 19.6 mm to (9.21, 32.1)
- moved U$2 8.90 mm to (47.0, 42.2)
- moved S5 6.35 mm to (67.3, 56.8), turned to 180 degrees
- moved S1 4.02 mm to (26.7, 26.7)
- moved S2 3.72 mm to (16.8, 26.7)
- moved S3 3.19 mm to (23.5, 57.5)
- moved U$1 2.84 mm to (58.4, 12.7)
- moved S4 0.71 mm to (31.1, 57.5)
- renumbered R1 to A2
Routing:
- net A1: track 88.7 -> 48.1 mm, vias 1 -> 0
- net SDA: track 149.4 -> 111.7 mm, vias 2 -> 1
- net SCL: track 146.8 -> 111.4 mm, vias 1 -> 2
- net LED2: track 22.2 -> 43.0 mm, vias 2 -> 0
- net SCK: track 61.4 -> 41.2 mm, vias 1 -> 0
- net MOSI: track 79.8 -> 61.2 mm, vias 0 -> 2
- net MISO: track 73.0 -> 59.5 mm, vias 0 -> 2
- net R3: track 40.8 -> 54.0 mm
- net T4: track 45.5 -> 34.4 mm
- net DP2: track 19.2 -> 8.58 mm
- net P2: track 79.5 -> 69.9 mm, vias 2 -> 0
- net T1: track 53.4 -> 60.7 mm
- net R2: track 101.7 -> 96.6 mm, vias 0 -> 3
- net C2: track 45.0 -> 47.5 mm, vias 1 -> 0
- net R4: track 28.7 -> 26.7 mm, vias 0 -> 1
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Other:
- board size 82.5 x 116.5 mm -> 83.2 x 116.5 mm
- board text added: "A1"
- board text added: "CS: 10"
- board text added: "I2C: 18,19"
- board text added: "MAIN 2"
- board text added: "MAIN 3"
- board text added: "MAIN TEENSY 4.1"
- board text added: "SECONDARY TEENSY 4.0"
- board text added: "Version 1.1 Benjamin Boeckman & Evan Sittauer"
- board text removed: "CS: Main 10"
- board text removed: "I2C: MAIN 18,19"
- board text removed: "MAIN DP2"
- board text removed: "MAIN DP3"
- board text removed: "MAIN TEENSY"
- board text removed: "Main17\"
- board text removed: "SECONDARY TEENSY"
- board text removed: "Version 1.0 Benjamin Boeckman"

Commit message: some changes
Parts:
- moved S4 17.2 mm to (48.3, 58.1)
- moved S3 10.2 mm to (33.7, 58.1)
Routing:
- net SCK: track 41.2 -> 77.1 mm
- net A1: track 48.1 -> 77.1 mm
- net R2: track 96.6 -> 73.9 mm, vias 3 -> 0
- net SDA: track 111.7 -> 133.7 mm, vias 1 -> 0
- net R3: track 54.0 -> 33.0 mm
- net R4: track 26.7 -> 10.9 mm, vias 1 -> 0
- net SCL: track 111.4 -> 124.4 mm, vias 2 -> 0
- net P2: track 69.9 -> 81.2 mm
- net T2: track 61.0 -> 72.1 mm
- net T4: track 34.4 -> 27.5 mm
- net T1: track 60.7 -> 66.2 mm, vias 2 -> 0
- net C2: track 47.5 -> 52.7 mm
- net T3: track 34.8 -> 30.0 mm
- net MOSI: track 61.2 -> 64.9 mm, vias 2 -> 0
- net LED2: track 43.0 -> 39.4 mm
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